Commit message: Componenets

File: asdesc/robots/base_only.xacro (robot description, xacro)
@@ -4,5 +4,4 @@
        xmlns:interface="http://playerstage.sourceforge.net/gazebo/xmlschema/#interface"
        xmlns:xacro="http://ros.org/wiki/xacro" name="asbase">
-      <xacro:include filename="$(find asdesc)/urdf/base/as_base.xacro" />
-      <xacro:as_base/>
+      <xacro:include filename="$(find asdesc)/urdf/base/asbase.xacro" />
 </robot>

File: asdesc/robots/basearm.xacro (robot description, xacro)
@@ -10,14 +10,11 @@
       <xacro:arg name="effort_control" default="false"/>
       <!-- includes -->
-      <xacro:include filename="$(find asdesc)/urdf/base/as_base.xacro" />
+      <xacro:include filename="$(find asdesc)/urdf/base/asbase.xacro" />
       <xacro:include filename="$(find xarm_description)/urdf/xarm6_robot_macro.xacro" />
       <!-- formation-->
-      <xacro:as_base/>
-      <xacro:xarm6_robot prefix="$(arg prefix)"
-            namespace="$(arg ros_namespace)"
-            limited="$(arg limited)"
-            effort_control="$(arg effort_control)"
-            attach_to="base_link"
-            xyz="${-0.15 + base_link_dx/2} 0 ${0.03-base_link_dz/2}"
-            rpy="0 0 0" />
+      <!-- <xacro:as_base/> -->
+      <xacro:xarm6_robot prefix="$(arg prefix)" namespace="$(arg ros_namespace)" limited="$(arg limited)" effort_control="$(arg effort_control)" attach_to="base_link" xyz="${-0.15 + base_link_dx/2} 0 ${0.03-base_link_dz/2}" rpy="0 0 0" />
+      <!-- <xacro:property name="extruder_parent" value=" 0 0 0"/>
+	<xacro:property name="extruder_xyz" value=" 0 0 0"/>
+	<xacro:property name="extruder_rpy" value="0.455"/> -->
 </robot>
