Commit message: renaming packages to as_ prefix

File: as_description/robots/base_only.xacro (robot description, xacro)
@@ -4,4 +4,4 @@
        xmlns:interface="http://playerstage.sourceforge.net/gazebo/xmlschema/#interface"
        xmlns:xacro="http://ros.org/wiki/xacro" name="asbase">
-      <xacro:include filename="$(find asdesc)/urdf/base/asbase.xacro" />
+      <xacro:include filename="$(find as_description)/urdf/base/asbase.xacro" />
 </robot>

File: as_description/robots/basearm.xacro (robot description, xacro)
@@ -10,5 +10,5 @@
       <xacro:arg name="effort_control" default="false"/>
       <!-- includes -->
-      <xacro:include filename="$(find asdesc)/urdf/base/asbase.xacro" />
+      <xacro:include filename="$(find as_description)/urdf/base/asbase.xacro" />
       <xacro:include filename="$(find xarm_description)/urdf/xarm6_robot_macro.xacro" />
       <!-- formation-->

File: as_description/urdf/base/as_base.xacro (robot description, xacro)
@@ -5,6 +5,46 @@
 	xmlns:xacro="http://ros.org/wiki/xacro">
 	<!-- Common -->
-	<xacro:include filename="$(find asdesc)/urdf/common/inertia.xacro"/>
-	<xacro:include filename="$(find asdesc)/urdf/common/materials.xacro"/>
+	<xacro:include filename="$(find as_description)/urdf/common/inertia.xacro"/>
+	<xacro:include filename="$(find as_description)/urdf/common/materials.xacro"/>
+	<!-- Link Dimensions -->
+	<!-- base_link -->
+	<xacro:property name="base_link_dx" value="0.8"/>
+	<xacro:property name="base_link_dy" value="0.5"/>
+	<xacro:property name="base_link_dz" value="0.2"/>
+	<xacro:property name="base_link_m" value="2"/>
+	<!-- alluminium frame only -->
+	<!-- wheel_link -->
+	<xacro:property name="wheel_link_r" value="${0.152/2}"/>
+	<xacro:property name="wheel_link_m" value="0.6"/>
+	<xacro:property name="wheel_roller_angle" value="${45*M_PI/180}"/>
+	<!-- motor_gearbox_link -->
+	<xacro:property name="motor_link_r" value="0.025"/>
+	<xacro:property name="motor_link_h" value="0.12"/>
+	<xacro:property name="motor_link_m" value="0.5"/>
+	<!-- True is 1460mNm -->
+	<xacro:property name="motor_effort_limit" value="1.4"/>
+	<!-- True is 6110rpm -->
+	<xacro:property name="motor_velocity_limit" value="600"/>
+	<xacro:property name="gearbox_reduction" value="91"/>
+	<!-- battery_link -->
+	<xacro:property name="battery_link_dx" value="0.8"/>
+	<xacro:property name="battery_link_dy" value="0.5"/>
+	<xacro:property name="battery_link_dz" value="0.2"/>
+	<xacro:property name="battery_link_m" value="6.7"/>
+	<!-- nuc_link -->
+	<xacro:property name="nuc_link_dx" value="0.12"/>
+	<xacro:property name="nuc_link_dy" value="0.12"/>
+	<xacro:property name="nuc_link_dz" value="0.06"/>
+	<xacro:property name="nuc_link_m" value="0.3"/>
+	<!-- offsets -->
+	<xacro:property name="motor_wheel_assemply_xyz_fl" value="0.375 0.25 -0.08"/>
+	<xacro:property name="motor_wheel_assemply_rpy_fl" value="${- M_PI/2} 0 0"/>
+	<xacro:property name="motor_wheel_assemply_xyz_fr" value="0.375 -0.25 -0.08"/>
+	<xacro:property name="motor_wheel_assemply_rpy_fr" value="${M_PI/2} 0 0"/>
+	<xacro:property name="motor_wheel_assemply_xyz_bl" value="-0.375 0.25 -0.08"/>
+	<xacro:property name="motor_wheel_assemply_rpy_bl" value="${ M_PI/2} 0 ${M_PI}"/>
+	<xacro:property name="motor_wheel_assemply_xyz_br" value="-0.375 -0.25 -0.08"/>
+	<xacro:property name="motor_wheel_assemply_rpy_br" value="${-M_PI/2} 0 ${M_PI}"/>
+	<xacro:property name="ground_clearance" value="0.05"/>
 	<xacro:macro name="as_motor_wheel_assembly" params="suffix">
 		<link name="motor_gearbox${suffix}">

File: as_description/urdf/base/asbase.xacro (robot description, xacro)
@@ -37,6 +37,6 @@
 	<xacro:property name="ground_clearance" value="${motor_link_r/2 +wheel_link_r/2}"/>
 	<!-- Import Things -->
-	<xacro:include filename="$(find asdesc)/urdf/base/chasis.xacro"/>
-	<xacro:include filename="$(find asdesc)/urdf/components/components.xacro"/>
+	<xacro:include filename="$(find as_description)/urdf/base/chasis.xacro"/>
+	<xacro:include filename="$(find as_description)/urdf/components/components.xacro"/>
 	<!-- Componenet positions-->
 	<xacro:property name="battery_xyz" value="-${base_link_dx/2 - 0.18} 0 -${base_link_dz/2 - 0.01 - battery_link_dz/2}"/>

File: as_description/urdf/base/chasis.xacro (robot description, xacro)
@@ -5,46 +5,6 @@
 	xmlns:xacro="http://ros.org/wiki/xacro">
 	<!-- Common -->
-	<xacro:include filename="$(find asdesc)/urdf/common/inertia.xacro"/>
-	<xacro:include filename="$(find asdesc)/urdf/common/materials.xacro"/>
-	<!-- Link Dimensions -->
-	<!-- base_link -->
-	<xacro:property name="base_link_dx" value="0.8"/>
-	<xacro:property name="base_link_dy" value="0.5"/>
-	<xacro:property name="base_link_dz" value="0.2"/>
-	<xacro:property name="base_link_m" value="2"/>
-	<!-- alluminium frame only -->
-	<!-- wheel_link -->
-	<xacro:property name="wheel_link_r" value="${0.152/2}"/>
-	<xacro:property name="wheel_link_m" value="0.6"/>
-	<xacro:property name="wheel_roller_angle" value="${45*M_PI/180}"/>
-	<!-- motor_gearbox_link -->
-	<xacro:property name="motor_link_r" value="0.025"/>
-	<xacro:property name="motor_link_h" value="0.12"/>
-	<xacro:property name="motor_link_m" value="0.5"/>
-	<!-- True is 1460mNm -->
-	<xacro:property name="motor_effort_limit" value="1.4"/>
-	<!-- True is 6110rpm -->
-	<xacro:property name="motor_velocity_limit" value="600"/>
-	<xacro:property name="gearbox_reduction" value="91"/>
-	<!-- battery_link -->
-	<xacro:property name="battery_link_dx" value="0.8"/>
-	<xacro:property name="battery_link_dy" value="0.5"/>
-	<xacro:property name="battery_link_dz" value="0.2"/>
-	<xacro:property name="battery_link_m" value="6.7"/>
-	<!-- nuc_link -->
-	<xacro:property name="nuc_link_dx" value="0.12"/>
-	<xacro:property name="nuc_link_dy" value="0.12"/>
-	<xacro:property name="nuc_link_dz" value="0.06"/>
-	<xacro:property name="nuc_link_m" value="0.3"/>
-	<!-- offsets -->
-	<xacro:property name="motor_wheel_assemply_xyz_fl" value="0.375 0.25 -0.08"/>
-	<xacro:property name="motor_wheel_assemply_rpy_fl" value="${- M_PI/2} 0 0"/>
-	<xacro:property name="motor_wheel_assemply_xyz_fr" value="0.375 -0.25 -0.08"/>
-	<xacro:property name="motor_wheel_assemply_rpy_fr" value="${M_PI/2} 0 0"/>
-	<xacro:property name="motor_wheel_assemply_xyz_bl" value="-0.375 0.25 -0.08"/>
-	<xacro:property name="motor_wheel_assemply_rpy_bl" value="${ M_PI/2} 0 ${M_PI}"/>
-	<xacro:property name="motor_wheel_assemply_xyz_br" value="-0.375 -0.25 -0.08"/>
-	<xacro:property name="motor_wheel_assemply_rpy_br" value="${-M_PI/2} 0 ${M_PI}"/>
-	<xacro:property name="ground_clearance" value="0.05"/>
+	<xacro:include filename="$(find as_description)/urdf/common/inertia.xacro"/>
+	<xacro:include filename="$(find as_description)/urdf/common/materials.xacro"/>
 	<xacro:macro name="as_motor_wheel_assembly" params="suffix">
 		<link name="motor_gearbox${suffix}">

File: as_description/urdf/components/components.xacro (robot description, xacro)
@@ -1,5 +1,5 @@
 <?xml version="1.0"?>
 <robot xmlns:xacro="http://ros.org/wiki/xacro">
-	<xacro:include filename="$(find asdesc)/urdf/common/generic_links.xacro"/>
+	<xacro:include filename="$(find as_description)/urdf/common/generic_links.xacro"/>
 	<!-- battery_link -->
 	<xacro:property name="battery_link_dx" value="0.35"/>
