Commit message: Fixed some meshes and lowered the footprint link

File: as_description/robots/as_base.xacro (robot description, xacro)
@@ -15,7 +15,4 @@
 	<xacro:property name="battery_xyz" value="${-base_link_dx/2 + battery_link_dx/2 -0.08} 0  ${-base_link_dz/2 +0.02 + battery_link_dz/2 }" />
 	<xacro:property name="battery_rpy" value="0 0 0" />
-	<!-- TODO dealwith nuc -->
-	<!-- <xacro:property name="nuc_xyz" value="${-base_link_dx/2 + battery_link_dx/2 } 0  ${-base_link_dz/2 +0.02 + battery_link_dz/2 }" />
-	<xacro:property name="nuc_rpy" value="0 0 0" /> -->
 	<!-- Import macros -->
 	<xacro:include filename="$(find as_description)/urdf/base/chasis.macro.xacro" />
@@ -24,5 +21,4 @@
 	<xacro:as_base_chasis />
 	<xacro:battery48 parent="base_link" xyz="${battery_xyz}" rpy="${battery_rpy}" />
-	<!-- <xacro:nuc parent="base_link" xyz="${nuc_xyz}" rpy="${nuc_rpy}" /> -->
 	<xacro:dc_box parent="base_link" xyz="${dc_box_xyz}" rpy="${dc_box_rpy}" />
 	<xacro:mount_plate parent="base_link" xyz="${mount_plate_xyz}" rpy="${mount_plate_rpy}" />

File: as_description/urdf/base/chasis.params.xacro (robot description, xacro)
@@ -4,5 +4,5 @@
 	xmlns:interface="http://playerstage.sourceforge.net/gazebo/xmlschema/#interface"
 	xmlns:xacro="http://ros.org/wiki/xacro">
-<!-- Link Dimensions -->
+	<!-- Link Dimensions -->
 	<!-- base_link -->
 	<xacro:property name="base_link_dx" value="0.72" />
@@ -21,5 +21,4 @@
 	<!-- motor_gearbox_link -->
 	<xacro:property name="motor_link_r" value="0.025" />
-	<!-- motor normal 12 cm. But with coupler +5cm -->
 	<xacro:property name="motor_link_h" value="${0.12+0.1}" />
 	<xacro:property name="motor_link_m" value="${0.14 +0.36}" />
@@ -42,4 +41,4 @@
 	<xacro:property name="motor_wheel_assembly_xyz_br" value="-${base_link_dx/2-0.077/2} -${base_link_dy/2 -motor_pad_l/2 - 0.025} -${base_link_dz/2 + motor_link_r/2 +0.012}" />
 	<xacro:property name="motor_wheel_assembly_rpy_br" value="${M_PI/2} 0 0" />
-	<xacro:property name="ground_clearance" value="${motor_link_r/2 +wheel_link_r/2}" />
+	<xacro:property name="ground_clearance" value="${0.012+ motor_link_r/2 +wheel_link_r}" />
 </robot>

File: as_description/urdf/base/components.macro.xacro (robot description, xacro)
@@ -35,9 +35,9 @@
 		<xacro:generic_box name="battery48" parent="${parent}" xyz="${xyz}" rpy="${rpy}" dx="${battery_link_dx}" dy="${battery_link_dy}" dz="${battery_link_dz}" m="${battery_link_m}" material="LightGrey" gmaterial="Gazebo/LightGrey" meshfile="battery.dae" mxyz="0.035 0 ${-battery_link_dz/2}" mrpy="0 0 ${M_PI}" />
 	</xacro:macro>
-	<xacro:macro name="nuc" params="parent xyz rpy">
-		<xacro:generic_box name="nuc" parent="${parent}" xyz="${xyz}" rpy="${rpy}" dx="${nuc_link_dx}" dy="${nuc_link_dy}" dz="${nuc_link_dz}" m="${nuc_link_m}" material="DarkGrey" gmaterial="Gazebo/DarkGrey" meshfile="" mxyz="" mrpy="" />
+	<xacro:macro name="nuc" params="parent xyz rpy suffix">
+		<xacro:generic_box name="nuc${suffix}" parent="${parent}" xyz="${xyz}" rpy="${rpy}" dx="${nuc_link_dx}" dy="${nuc_link_dy}" dz="${nuc_link_dz}" m="${nuc_link_m}" material="DarkGrey" gmaterial="Gazebo/DarkGrey" meshfile="nuc.stl" mxyz="0 0 0" mrpy="0 0 0" />
 	</xacro:macro>
 	<xacro:macro name="dc_box" params="parent xyz rpy">
-		<xacro:generic_box name="dc_box" parent="${parent}" xyz="${xyz}" rpy="${rpy}" dx="${dc_box_dx}" dy="${dc_box_dy}" dz="${dc_box_dz}" m="${dc_box_m}" material="LightGrey" gmaterial="Gazebo/LightGrey" meshfile="dcbox.stl" mxyz="0 ${-dc_box_dx/2} 0" mrpy="0 ${M_PI/2} ${M_PI/2}" />
+		<xacro:generic_box name="dc_box" parent="${parent}" xyz="${xyz}" rpy="${rpy}" dx="${dc_box_dx}" dy="${dc_box_dy}" dz="${dc_box_dz}" m="${dc_box_m}" material="LightGrey" gmaterial="Gazebo/LightGrey" meshfile="dcbox.dae" mxyz="0 0 ${dc_box_dz/2}" mrpy="0 0 ${M_PI/2} " />
 	</xacro:macro>
 	<xacro:macro name="mount_plate" params="parent xyz rpy">

Commit message: WIP gazebo
 loading second gazebo control messes up the first one.  making arm collapse. also base wheel directions are wrong. change.

File: as_description/robots/as_base.xacro (robot description, xacro)
@@ -25,3 +25,11 @@
 	<!-- <xacro:compressor parent="base_link" xyz="${compressor_xyz}" rpy="${compressor_rpy}" /> -->
 	<!-- <xacro:material3 parent="base_link" xyz="${material3_xyz}" rpy="${material3_rpy}" /> -->
+	<!-- gazebo_plugin -->
+	<!-- <xacro:if value="${load_gazebo_plugin}"> -->
+		<gazebo>
+			<plugin name="gazebo_ros_control" filename="libgazebo_ros_control.so">
+				<robotNamespace>/as_base</robotNamespace>
+			</plugin>
+		</gazebo>
+	<!-- </xacro:if> -->
 </robot>

File: as_description/urdf/base/chasis.macro.xacro (robot description, xacro)
@@ -7,5 +7,5 @@
 	<xacro:include filename="$(find as_description)/urdf/common/inertia.xacro"/>
 	<xacro:include filename="$(find as_description)/urdf/common/materials.xacro"/>
-	<xacro:macro name="as_motor_wheel_assembly" params="suffix wheel_angle" >
+	<xacro:macro name="as_motor_wheel_assembly" params="suffix wheel_angle  " >
 		<link name="motor_gearbox${suffix}">
 			<inertial>
@@ -32,5 +32,5 @@
 			<axis xyz="0 0 1"/>
 			<limit effort = "${motor_effort_limit}" velocity = "${motor_velocity_limit}" />
-			<!-- <dynamics damping="1.5"/> -->
+			<dynamics damping="1.5" friction="1.0"/>
 		</joint>
 		<transmission name="motor_wheel_joint_transmission${suffix}">
@@ -48,5 +48,5 @@
 				<origin xyz="0 0 0" rpy="0 0 0"/>
 				<mass value="${wheel_link_m}"/>
-				<xacro:sphere_inertia_tensor m="${wheel_link_m}" r="${wheel_link_r}" />
+				<xacro:sphere_inertia_tensor m="${wheel_link_m}" r="${wheel_link_r/2}" />
 			</inertial>
 			<!-- No visual. -->
@@ -134,9 +134,4 @@
 			<origin xyz= "${motor_wheel_assembly_xyz_br}" rpy = "${motor_wheel_assembly_rpy_br}" />
 		</joint>
-		<gazebo>
-			<plugin name="gazebo_ros_control" filename="libgazebo_ros_control.so">
-				<robotNamespace>/as_base</robotNamespace>
-			</plugin>
-		</gazebo>
 	</xacro:macro>
 </robot>

File: as_description/urdf/base/chasis.params.xacro (robot description, xacro)
@@ -28,8 +28,9 @@
 	<xacro:property name="motor_meshfile" value="motor.dae" />
 	<!-- True is 1460mNm -->
-	<xacro:property name="motor_effort_limit" value="1" />
+	<xacro:property name="motor_effort_limit" value="50" />
 	<!-- True is 6110rpm. Which is 7.031 rad/s I think. So 5 to be safe.-->
 	<xacro:property name="motor_velocity_limit" value="5" />
-	<xacro:property name="gearbox_reduction" value="91" />
+	<!-- <xacro:property name="gearbox_reduction" value="91" /> -->
+	<xacro:property name="gearbox_reduction" value="1" />
 	<!-- offsets -->
 	<xacro:property name="motor_wheel_assembly_xyz_fl" value="${base_link_dx/2-0.077/2} ${base_link_dy/2 -motor_pad_l/2 - 0.025} -${base_link_dz/2 + motor_link_r/2 +0.012}" />
