Commit message: changed chasis collision box. and creeated new generated urdf

File: as_description/robots/as.generated.urdf (robot description, URDF)
Before this commit: robot armstone, 25 links, 24 joints
Links:
- added link backpack_link; collision box size=0.4 0.4 0.18
- added link base_imu_frame
- added link base_imu_module; visual box size=0.025 0.025 0.0075
- added link compressor_link, mass 1.1; collision box size=0.242 0.055 0.12; visual mesh filename=package://as_description/meshes/compressor_assembly.dae
- added link cover_plate_link, mass 0.2; collision box size=0.47 0.45 0.006; visual mesh filename=package://as_description/meshes/cover_assembly_.dae
- added link ee_imu_frame
- added link ee_imu_module; visual box size=0.025 0.025 0.0075
- added link ic_link, mass 0.4; collision box size=0.28 0.074 0.145; visual mesh filename=package://as_description/meshes/intermediate_assembly.dae
- added link material3_link, mass 5.28; collision cylinder length=0.42 radius=0.0525; visual mesh filename=package://as_description/meshes/clay_assembly.dae
- link base_link: geometry collision box size=0.025 0.025 0.29; collision box size=0.025 0.025 0.29
Joints:
- added joint backpack_joint: type fixed, parent base_link, child backpack_link, origin xyz=-0.16 0  0.176 rpy=0 0 0
- added joint base_imu_module_joint1: type fixed, parent base_link, child base_imu_module, origin xyz=-0.0125 0  0.066 rpy=0 0 0
- added joint base_imu_module_joint2: type fixed, parent base_imu_module, child base_imu_frame, origin xyz= 0.007 0 0 rpy=0 0 0
- added joint compressor_joint: type fixed, parent base_link, child compressor_link, origin xyz=-0.239 0.1287 0.146 rpy=0 0 0
- added joint cover_plate_joint: type fixed, parent base_link, child cover_plate_link, origin xyz=-0.125 0 0.086 rpy=0 0 0
- added joint ee_imu_module_joint1: type fixed, parent xarmlink_eef, child ee_imu_module, origin xyz=0 -0.06125 0 rpy=0 3.14159265359 0
- added joint ee_imu_module_joint2: type fixed, parent ee_imu_module, child ee_imu_frame, origin xyz= 0.007 0 0 rpy=0 0 0
- added joint ic_joint: type fixed, parent base_link, child ic_link, origin xyz=-0.235 -0.1505  0.1585 rpy=0 0 0
- added joint material3_joint: type fixed, parent base_link, child material3_link, origin xyz=-0.209 0 0.1585 rpy=0 1.57079632679 0

File: as_description/urdf/base/chasis.macro.xacro (robot description, xacro)
@@ -106,6 +106,25 @@
 			</visual>
 			<collision>
+				<origin xyz= "-0.125 0 0" rpy = "0 0 0" />
 				<geometry>
-					<box size="${base_link_dx} ${base_link_dy} ${base_link_dz}" />
+					<box size="${base_link_dx-0.25} ${base_link_dy} ${base_link_dz}" />
+				</geometry>
+			</collision>
+			<collision>
+				<origin xyz= "0 0 ${-(base_link_dz-0.03)/2}" rpy = "0 0 0" />
+				<geometry>
+					<box size="${base_link_dx} ${base_link_dy} 0.035" />
+				</geometry>
+			</collision>
+			<collision>
+				<origin xyz= "${base_link_dx/2 -0.125} ${base_link_dy/2 -0.01} 0.015" rpy = "0 ${-60*M_PI/180} 0" />
+				<geometry>
+					<box size=" 0.025 0.025 0.29" />
+				</geometry>
+			</collision>
+			<collision>
+				<origin xyz= "${base_link_dx/2 -0.125} ${-base_link_dy/2 +0.01} 0.015" rpy = "0 ${-60*M_PI/180} 0" />
+				<geometry>
+					<box size=" 0.025 0.025 0.29" />
 				</geometry>
 			</collision>
