Commit message: WIP towards cleaned up description and gazebo stack

File: as_description/robots/as.xacro (robot description, xacro)
@@ -1,6 +1,19 @@
 <?xml version="1.0"?>
 <robot xmlns:sensor="http://playerstage.sourceforge.net/gazebo/xmlschema/#sensor"
-       xmlns:controller="http://playerstage.sourceforge.net/gazebo/xmlschema/#controller"
-       xmlns:interface="http://playerstage.sourceforge.net/gazebo/xmlschema/#interface"
-       xmlns:xacro="http://ros.org/wiki/xacro" >
+      xmlns:controller="http://playerstage.sourceforge.net/gazebo/xmlschema/#controller"
+      xmlns:interface="http://playerstage.sourceforge.net/gazebo/xmlschema/#interface"
+      xmlns:xacro="http://ros.org/wiki/xacro" name="armstone">
+      <!-- Arm arguments -->
+      <xacro:arg name="prefix" default="xarm"/>
+      <xacro:arg name="ros_namespace" default="xarm"/>
+      <xacro:arg name="limited" default="true"/>
+      <xacro:arg name="effort_control" default="false"/>
+      <!-- includes -->
+      <xacro:include filename="$(find xarm_description)/urdf/xarm6_robot_macro.xacro" />
+      <!-- formation-->
+      <xacro:include filename="$(find as_description)/robots/as_base.xacro" />
+      <xacro:xarm6_robot prefix="$(arg prefix)" namespace="$(arg ros_namespace)" limited="$(arg limited)" effort_control="$(arg effort_control)" attach_to="base_link" xyz="${-0.15 + base_link_dx/2} 0 ${0.03-base_link_dz/2}" rpy="0 0 0" />
+      <!-- <xacro:property name="extruder_parent" value=" 0 0 0"/>
+	<xacro:property name="extruder_xyz" value=" 0 0 0"/>
+	<xacro:property name="extruder_rpy" value="0.455"/> -->
 </robot>

File: as_description/urdf/base/chasis.macro.xacro (robot description, xacro)
@@ -7,5 +7,5 @@
 	<xacro:include filename="$(find as_description)/urdf/common/inertia.xacro"/>
 	<xacro:include filename="$(find as_description)/urdf/common/materials.xacro"/>
-	<xacro:macro name="as_motor_wheel_assembly" params="suffix">
+	<xacro:macro name="as_motor_wheel_assembly" params="suffix wheel_angle" >
 		<link name="motor_gearbox${suffix}">
 			<inertial>
@@ -15,8 +15,8 @@
 			</inertial>
 			<visual>
+				<origin xyz= "${motor_mxyz}" rpy = "${motor_mrpy}" />
 				<geometry>
-					<cylinder length="${motor_link_h}" radius="${motor_link_r}"/>
+					<mesh filename="package://as_description/meshes/${motor_meshfile}" />
 				</geometry>
-				<material name="BlackClear"/>
 			</visual>
 			<collision>
@@ -29,5 +29,5 @@
 			<parent link="motor_gearbox${suffix}"/>
 			<child link="omniwheel${suffix}"/>
-			<origin xyz= "0 0 ${motor_link_h/2}" rpy = "0 ${wheel_roller_angle} 0" />
+			<origin xyz= "0 0 ${motor_link_h/2}" rpy = "0 ${wheel_angle} 0" />
 			<axis xyz="0 0 1"/>
 			<limit effort = "${motor_effort_limit}" velocity = "${motor_velocity_limit}" />
@@ -50,10 +50,5 @@
 				<xacro:sphere_inertia_tensor m="${wheel_link_m}" r="${wheel_link_r}" />
 			</inertial>
-			<visual>
-				<geometry>
-					<cylinder radius="${wheel_link_r}" length="0.05"/>
-				</geometry>
-				<material name="WhiteClear"/>
-			</visual>
+			<!-- No visual. -->
 			<collision>
 				<geometry>
@@ -95,8 +90,8 @@
 			</inertial>
 			<visual>
+				<origin xyz= "${base_mxyz}" rpy = "${base_mrpy}" />
 				<geometry>
-					<box size="${base_link_dx} ${base_link_dy} ${base_link_dz}" />
+					<mesh filename="package://as_description/meshes/${base_meshfile}" />
 				</geometry>
-				<material name="DarkGreyClear"/>
 			</visual>
 			<collision>
@@ -109,8 +104,8 @@
 			</gazebo>
 		</link>
-		<xacro:as_motor_wheel_assembly suffix="_fl"/>
-		<xacro:as_motor_wheel_assembly suffix="_fr"/>
-		<xacro:as_motor_wheel_assembly suffix="_bl"/>
-		<xacro:as_motor_wheel_assembly suffix="_br"/>
+		<xacro:as_motor_wheel_assembly suffix="_fl"  wheel_angle="${-wheel_roller_angle}"/>
+		<xacro:as_motor_wheel_assembly suffix="_fr"  wheel_angle="${wheel_roller_angle}"/>
+		<xacro:as_motor_wheel_assembly suffix="_bl"  wheel_angle="${wheel_roller_angle}"/>
+		<xacro:as_motor_wheel_assembly suffix="_br"  wheel_angle="${-wheel_roller_angle}"/>
 		<joint name="motor_wheel_assembly_joint_fl" type="fixed">
 			<parent link="base_link"/>

File: as_description/urdf/base/chasis.params.xacro (robot description, xacro)
@@ -11,4 +11,7 @@
 	<!-- 2.8kg raw frame. 3.5 estimate  full -->
 	<xacro:property name="base_link_m" value="3.5" />
+	<xacro:property name="base_meshfile" value="chasis.dae" />
+	<xacro:property name="base_mxyz" value="${(base_link_dx/2 - 0.01)} 0 ${(0.02 - 0.006 -base_link_dz/2)}" />
+	<xacro:property name="base_mrpy" value="0 0 0" />
 	<!-- alluminium frame only -->
 	<!-- wheel_link -->
@@ -19,6 +22,10 @@
 	<xacro:property name="motor_link_r" value="0.025" />
 	<!-- motor normal 12 cm. But with coupler +5cm -->
-	<xacro:property name="motor_link_h" value="${0.12+0.05}" />
+	<xacro:property name="motor_link_h" value="${0.12+0.1}" />
 	<xacro:property name="motor_link_m" value="${0.14 +0.36}" />
+	<xacro:property name="motor_pad_l" value="0.0931" />
+	<xacro:property name="motor_mrpy" value="${M_PI/2} ${- M_PI/2} 0" />
+	<xacro:property name="motor_mxyz" value="0 ${motor_link_r/2 +0.012} 0.025" />
+	<xacro:property name="motor_meshfile" value="motor.dae" />
 	<!-- True is 1460mNm -->
 	<xacro:property name="motor_effort_limit" value="1" />
@@ -27,12 +34,12 @@
 	<xacro:property name="gearbox_reduction" value="91" />
 	<!-- offsets -->
-	<xacro:property name="motor_wheel_assembly_xyz_fl" value="${base_link_dx/2-0.035} ${base_link_dy/2 -motor_link_h/2} -${base_link_dz/2 + motor_link_r/2}" />
-	<xacro:property name="motor_wheel_assembly_rpy_fl" value="${- M_PI/2} 0 0" />
-	<xacro:property name="motor_wheel_assembly_xyz_fr" value="${base_link_dx/2-0.035} -${base_link_dy/2 -motor_link_h/2} -${base_link_dz/2 + motor_link_r/2}" />
+	<xacro:property name="motor_wheel_assembly_xyz_fl" value="${base_link_dx/2-0.077/2} ${base_link_dy/2 -motor_pad_l/2 - 0.025} -${base_link_dz/2 + motor_link_r/2 +0.012}" />
+	<xacro:property name="motor_wheel_assembly_rpy_fl" value="${M_PI/2} 0 ${M_PI}" />
+	<xacro:property name="motor_wheel_assembly_xyz_fr" value="${base_link_dx/2-0.077/2} -${base_link_dy/2 -motor_pad_l/2 - 0.025} -${base_link_dz/2 + motor_link_r/2 +0.012}" />
 	<xacro:property name="motor_wheel_assembly_rpy_fr" value="${M_PI/2} 0 0" />
-	<xacro:property name="motor_wheel_assembly_xyz_bl" value="-${base_link_dx/2-0.035} ${base_link_dy/2 -motor_link_h/2} -${base_link_dz/2 + motor_link_r/2}" />
+	<xacro:property name="motor_wheel_assembly_xyz_bl" value="-${base_link_dx/2-0.077/2} ${base_link_dy/2 -motor_pad_l/2 - 0.025} -${base_link_dz/2 + motor_link_r/2 +0.012}" />
 	<xacro:property name="motor_wheel_assembly_rpy_bl" value="${ M_PI/2} 0 ${M_PI}" />
-	<xacro:property name="motor_wheel_assembly_xyz_br" value="-${base_link_dx/2-0.035} -${base_link_dy/2 -motor_link_h/2} -${base_link_dz/2 + motor_link_r/2}" />
-	<xacro:property name="motor_wheel_assembly_rpy_br" value="${-M_PI/2} 0 ${M_PI}" />
+	<xacro:property name="motor_wheel_assembly_xyz_br" value="-${base_link_dx/2-0.077/2} -${base_link_dy/2 -motor_pad_l/2 - 0.025} -${base_link_dz/2 + motor_link_r/2 +0.012}" />
+	<xacro:property name="motor_wheel_assembly_rpy_br" value="${M_PI/2} 0 0" />
 	<xacro:property name="ground_clearance" value="${motor_link_r/2 +wheel_link_r/2}" />
 </robot>

File: as_description/urdf/base/components.macro.xacro (robot description, xacro)
@@ -3,7 +3,7 @@
 	<xacro:include filename="$(find as_description)/urdf/common/generic_links.xacro"/>
 	<!-- battery_link -->
-	<xacro:property name="battery_link_dx" value="0.35"/>
-	<xacro:property name="battery_link_dy" value="0.130"/>
-	<xacro:property name="battery_link_dz" value="0.082"/>
+	<xacro:property name="battery_link_dx" value="0.40"/>
+	<xacro:property name="battery_link_dy" value="0.150"/>
+	<xacro:property name="battery_link_dz" value="0.085"/>
 	<xacro:property name="battery_link_m" value="6.7"/>
 	<!-- nuc_link -->
@@ -22,5 +22,5 @@
 	<xacro:property name="material3_m" value="${3*1760/1000}"/>
 	<!-- Aluminium plate -->
-	<xacro:property name="mount_plate_dx" value="${0.72/2}"/>
+	<xacro:property name="mount_plate_dx" value="${0.27}"/>
 	<xacro:property name="mount_plate_dy" value="${0.455}"/>
 	<xacro:property name="mount_plate_dz" value="0.008"/>
@@ -32,30 +32,21 @@
 	<xacro:property name="compressor_h" value="0.13"/>
 	<xacro:property name="compressor_m" value="1.4"/>
-	<!-- Extruder -->
-	<xacro:property name="extruder_r" value="0.05"/>
-	<xacro:property name="extruder_h" value="0.18"/>
-	<!--Without material m 0.8  -->
-	<xacro:property name="extruder_m" value="1.5"/>
 	<xacro:macro name="battery48" params="parent xyz rpy">
-		<xacro:generic_box name="battery48" parent="${parent}" xyz="${xyz}" rpy="${rpy}" dx="${battery_link_dx}" dy="${battery_link_dy}" dz="${battery_link_dz}" m="${battery_link_m}" material="LightGrey" gmaterial="Gazebo/LightGrey" />
+		<xacro:generic_box name="battery48" parent="${parent}" xyz="${xyz}" rpy="${rpy}" dx="${battery_link_dx}" dy="${battery_link_dy}" dz="${battery_link_dz}" m="${battery_link_m}" material="LightGrey" gmaterial="Gazebo/LightGrey" meshfile="battery.dae" mxyz="0.035 0 ${-battery_link_dz/2}" mrpy="0 0 ${M_PI}" />
 	</xacro:macro>
 	<xacro:macro name="nuc" params="parent xyz rpy">
-		<xacro:generic_box name="nuc" parent="${parent}" xyz="${xyz}" rpy="${rpy}" dx="${nuc_link_dx}" dy="${nuc_link_dy}" dz="${nuc_link_dz}" m="${nuc_link_m}" material="DarkGrey" gmaterial="Gazebo/DarkGrey" />
+		<xacro:generic_box name="nuc" parent="${parent}" xyz="${xyz}" rpy="${rpy}" dx="${nuc_link_dx}" dy="${nuc_link_dy}" dz="${nuc_link_dz}" m="${nuc_link_m}" material="DarkGrey" gmaterial="Gazebo/DarkGrey" meshfile="" mxyz="" mrpy="" />
 	</xacro:macro>
 	<xacro:macro name="dc_box" params="parent xyz rpy">
-		<xacro:generic_box name="dc_box" parent="${parent}" xyz="${xyz}" rpy="${rpy}" dx="${dc_box_dx}" dy="${dc_box_dy}" dz="${dc_box_dz}" m="${dc_box_m}" material="Orange" gmaterial="Gazebo/Orange" />
+		<xacro:generic_box name="dc_box" parent="${parent}" xyz="${xyz}" rpy="${rpy}" dx="${dc_box_dx}" dy="${dc_box_dy}" dz="${dc_box_dz}" m="${dc_box_m}" material="LightGrey" gmaterial="Gazebo/LightGrey" meshfile="dcbox.stl" mxyz="0 ${-dc_box_dx/2} 0" mrpy="0 ${M_PI/2} ${M_PI/2}" />
 	</xacro:macro>
 	<xacro:macro name="mount_plate" params="parent xyz rpy">
-		<xacro:generic_box name="mount_plate" parent="${parent}" xyz="${xyz}" rpy="${rpy}" dx="${mount_plate_dx}" dy="${mount_plate_dy}" dz="${mount_plate_dz}" m="${mount_plate_m}" material="LightGrey" gmaterial="Gazebo/LightGrey" />
+		<xacro:generic_box name="mount_plate" parent="${parent}" xyz="${xyz}" rpy="${rpy}" dx="${mount_plate_dx}" dy="${mount_plate_dy}" dz="${mount_plate_dz}" m="${mount_plate_m}" material="LightGrey" gmaterial="Gazebo/LightGrey" meshfile="mounting_plate.stl" mxyz="0 0 ${-mount_plate_dz/2}" mrpy="0 0 ${M_PI/2}" />
 	</xacro:macro>
 	<xacro:macro name="compressor" params="parent xyz rpy">
-		<xacro:generic_cylinder name="compressor" parent="${parent}" xyz="${xyz}" rpy="${rpy}" r="${compressor_r}" h="${compressor_h}" m="${compressor_m}" material="Grey" gmaterial="Gazebo/Grey" />
-	</xacro:macro>
-	<!-- Extruder should not be macro. Probably own file -->
-	<xacro:macro name="extruder" params="parent xyz rpy">
-		<xacro:generic_cylinder name="extruder" parent="${parent}" xyz="${xyz}" rpy="${rpy}" r="${extruder_r}" h="${extruder_h}" m="${extruder_m}" material="Red" gmaterial="Gazebo/Red" />
+		<xacro:generic_cylinder name="compressor" parent="${parent}" xyz="${xyz}" rpy="${rpy}" r="${compressor_r}" h="${compressor_h}" m="${compressor_m}" material="Grey" gmaterial="Gazebo/Grey" meshfile="" mxyz="" mrpy="" />
 	</xacro:macro>
 	<xacro:macro name="material3" params="parent xyz rpy">
-		<xacro:generic_cylinder name="material3" parent="${parent}" xyz="${xyz}" rpy="${rpy}" r="${material3_r}" h="${material3_h}" m="${material3_m}" material="LightGrey" gmaterial="Gazebo/LightGrey" />
+		<xacro:generic_cylinder name="material3" parent="${parent}" xyz="${xyz}" rpy="${rpy}" r="${material3_r}" h="${material3_h}" m="${material3_m}" material="LightGrey" gmaterial="Gazebo/LightGrey" meshfile="" mxyz="" mrpy=""/>
 	</xacro:macro>
 </robot>

File: as_description/urdf/base/components.params.xacro (robot description, xacro)
@@ -32,8 +32,3 @@
 	<xacro:property name="compressor_h" value="0.13"/>
 	<xacro:property name="compressor_m" value="1.4"/>
-	<!-- Extruder -->
-	<xacro:property name="extruder_r" value="0.05"/>
-	<xacro:property name="extruder_h" value="0.18"/>
-	<!--Without material m 0.8  -->
-	<xacro:property name="extruder_m" value="1.5"/>
 </robot>

File: as_description/urdf/common/generic_links.xacro (robot description, xacro)
@@ -1,5 +1,5 @@
 <?xml version="1.0"?>
 <robot xmlns:xacro="http://ros.org/wiki/xacro">
-    <xacro:macro name="generic_box" params="parent name xyz rpy dx dy dz m material gmaterial">
+    <xacro:macro name="generic_box" params="parent name xyz rpy dx dy dz m material gmaterial meshfile mxyz mrpy">
         <joint name="${name}_joint" type="fixed">
             <parent link="${parent}"/>
@@ -14,7 +14,15 @@
             </inertial>
             <visual>
-                <geometry>
-                    <box size="${dx} ${dy} ${dz}" />
-                </geometry>
+                <xacro:if value="${len(meshfile)==0}">
+                    <geometry>
+                        <box size="${dx} ${dy} ${dz}" />
+                    </geometry>
+                </xacro:if>
+                <xacro:unless value="${len(meshfile)==0}">
+                    <origin xyz= "${mxyz}" rpy = "${mrpy}" />
+                    <geometry>
+                        <mesh filename="package://as_description/meshes/${meshfile}" />
+                    </geometry>
+                </xacro:unless>
                 <material name="${material}"/>
             </visual>
@@ -29,5 +37,5 @@
         </gazebo>
     </xacro:macro>
-    <xacro:macro name="generic_cylinder" params="parent name xyz rpy r h m material gmaterial">
+    <xacro:macro name="generic_cylinder" params="parent name xyz rpy r h m material gmaterial meshfile mxyz mrpy">
         <joint name="${name}_joint" type="fixed">
             <parent link="${parent}"/>
@@ -42,7 +50,15 @@
             </inertial>
             <visual>
-                <geometry>
-                    <cylinder radius="${r}" length="${h}" />
-                </geometry>
+                <xacro:if value="${len(meshfile)==0}">
+                    <geometry>
+                        <cylinder radius="${r}" length="${h}" />
+                    </geometry>
+                </xacro:if>
+                <xacro:unless value="${len(meshfile)==0}">
+                    <origin xyz= "${mxyz}" rpy = "${mrpy}" />
+                    <geometry>
+                        <mesh filename="package://as_description/meshes/${meshfile}" />
+                    </geometry>
+                </xacro:unless>
                 <material name="${material}"/>
             </visual>

Commit message: description updated launch files working

File: as_description/robots/as.xacro (robot description, xacro)
@@ -4,4 +4,5 @@
       xmlns:interface="http://playerstage.sourceforge.net/gazebo/xmlschema/#interface"
       xmlns:xacro="http://ros.org/wiki/xacro" name="armstone">
+      <xacro:include filename="$(find as_description)/urdf/base/chasis.params.xacro" />
       <!-- Arm arguments -->
       <xacro:arg name="prefix" default="xarm"/>
@@ -9,11 +10,14 @@
       <xacro:arg name="limited" default="true"/>
       <xacro:arg name="effort_control" default="false"/>
+      <xacro:arg name="velocity_control" default="false"/>
+      <xacro:property name="arm_xyz" value="${-0.185+base_link_dx/2} 0 ${0.005+0.028-base_link_dz/2}"/>
+      <xacro:property name="arm_rpy" value="0 0 0"/>
+      <xacro:property name="extruder_xyz" value="0 0 ${extruder_h/2}"/>
+      <xacro:property name="extruder_rpy" value="0 0 ${-M_PI/2}"/>
       <!-- includes -->
       <xacro:include filename="$(find xarm_description)/urdf/xarm6_robot_macro.xacro" />
       <!-- formation-->
       <xacro:include filename="$(find as_description)/robots/as_base.xacro" />
-      <xacro:xarm6_robot prefix="$(arg prefix)" namespace="$(arg ros_namespace)" limited="$(arg limited)" effort_control="$(arg effort_control)" attach_to="base_link" xyz="${-0.15 + base_link_dx/2} 0 ${0.03-base_link_dz/2}" rpy="0 0 0" />
-      <!-- <xacro:property name="extruder_parent" value=" 0 0 0"/>
-	<xacro:property name="extruder_xyz" value=" 0 0 0"/>
-	<xacro:property name="extruder_rpy" value="0.455"/> -->
+      <xacro:xarm6_robot prefix="$(arg prefix)" namespace="$(arg ros_namespace)" limited="$(arg limited)" effort_control="$(arg effort_control)" velocity_control="$(arg velocity_control)" attach_to="base_link" xyz="${arm_xyz}" rpy="${arm_rpy}" />
+      <xacro:extruder parent="xarmlink_eef" xyz="${extruder_xyz}" rpy="${extruder_rpy}" />
 </robot>

File: as_description/urdf/base/components.macro.xacro (robot description, xacro)
@@ -32,4 +32,10 @@
 	<xacro:property name="compressor_h" value="0.13"/>
 	<xacro:property name="compressor_m" value="1.4"/>
+	<!-- Extruder -->
+	<xacro:property name="extruder_r" value="0.05"/>
+    <xacro:property name="extruder_h" value="0.17"/>
+    <!--Without material m 1.05 (including bolts)  -->
+	<!--with tube maybe more-->
+    <xacro:property name="extruder_m" value="1.05"/>
 	<xacro:macro name="battery48" params="parent xyz rpy">
 		<xacro:generic_box name="battery48" parent="${parent}" xyz="${xyz}" rpy="${rpy}" dx="${battery_link_dx}" dy="${battery_link_dy}" dz="${battery_link_dz}" m="${battery_link_m}" material="LightGrey" gmaterial="Gazebo/LightGrey" meshfile="battery.dae" mxyz="0.035 0 ${-battery_link_dz/2}" mrpy="0 0 ${M_PI}" />
@@ -50,3 +56,44 @@
 		<xacro:generic_cylinder name="material3" parent="${parent}" xyz="${xyz}" rpy="${rpy}" r="${material3_r}" h="${material3_h}" m="${material3_m}" material="LightGrey" gmaterial="Gazebo/LightGrey" meshfile="" mxyz="" mrpy=""/>
 	</xacro:macro>
+	<xacro:macro name="extruder" params="parent xyz rpy">
+		<joint name="extruder_joint" type="fixed">
+            <parent link="${parent}"/>
+            <child link="extruder_link"/>
+            <origin xyz= "${xyz}" rpy = "${rpy}" />
+        </joint>
+        <link name="extruder_link">
+            <inertial>
+                <origin xyz="0 0 0" rpy="0 0 0"/>
+                <mass value="${extruder_m}"/>
+                <xacro:cylinder_inertia_tensor m="${extruder_m}" r="${extruder_r}" h="${extruder_h}"/>
+            </inertial>
+            <visual>
+				<origin xyz= "0 0 ${-extruder_h/2}" rpy = "0 0 0" />
+				<geometry>
+					<mesh filename="package://as_description/meshes/extruder.dae" />
+				</geometry>
+                <material name="Red"/>
+            </visual>
+            <collision>
+                <geometry>
+                    <cylinder radius="${extruder_r}" length="${extruder_h}" />
+                </geometry>
+            </collision>
+			<collision>
+				<origin xyz= "0 0 ${-extruder_h/2}" rpy = "0 0 0" />
+                <geometry>
+                    <cylinder radius="${extruder_r*1.5}" length="${extruder_h/2}" />
+                </geometry>
+            </collision>
+        </link>
+		<gazebo reference="extruder_link">
+            <material>Gazebo/Red</material>
+        </gazebo>
+		<link name="extruder_ee"/>
+		<joint name="extruder_ee_joint" type="fixed">
+			  <parent link="extruder_link"/>
+			  <child link="extruder_ee"/>
+			  <origin xyz= "0 0 ${extruder_h/2}" rpy = "0 0 0" />
+		</joint>
+	</xacro:macro>
 </robot>
