Commit message: WIP: holonomy done ! but not cleaned up stack

File: as_description/robots/as.xacro (robot description, xacro)
@@ -1,26 +1,31 @@
 <?xml version="1.0"?>
-<robot xmlns:sensor="http://playerstage.sourceforge.net/gazebo/xmlschema/#sensor"
-      xmlns:controller="http://playerstage.sourceforge.net/gazebo/xmlschema/#controller"
-      xmlns:interface="http://playerstage.sourceforge.net/gazebo/xmlschema/#interface"
-      xmlns:xacro="http://ros.org/wiki/xacro" name="armstone">
-      <xacro:include filename="$(find as_description)/urdf/base/chasis.params.xacro" />
+<robot xmlns:sensor="http://playerstage.sourceforge.net/gazebo/xmlschema/#sensor" xmlns:controller="http://playerstage.sourceforge.net/gazebo/xmlschema/#controller" xmlns:interface="http://playerstage.sourceforge.net/gazebo/xmlschema/#interface" xmlns:xacro="http://ros.org/wiki/xacro" name="armstone">
+      <!-- includes -->
+      <xacro:include filename="$(find xarm_description)/urdf/xarm6_robot_macro.xacro" />
+      <xacro:include filename="$(find as_description)/urdf/base/as_base.macro.xacro" />
       <!-- Arm arguments -->
       <!-- XARM -->
-      <xacro:arg name="prefix" default="xarm"/>
-      <xacro:arg name="ros_namespace" default="xarm"/>
-      <xacro:arg name="limited" default="true"/>
-      <xacro:arg name="effort_control" default="false"/>
-      <xacro:arg name="velocity_control" default="false"/>
-      <xacro:arg name="load_gazebo_plugin" default="false"/>
+      <xacro:arg name="prefix" default="xarm" />
+      <xacro:arg name="ros_namespace" default="/xarm" />
+      <xacro:arg name="limited" default="true" />
+      <xacro:arg name="effort_control" default="false" />
+      <xacro:arg name="velocity_control" default="false" />
+      <xacro:arg name="load_gazebo_plugin" default="false" />
       <!-- placement -->
-      <xacro:property name="arm_xyz" value="${-0.185+base_link_dx/2} 0 ${0.005+0.028-base_link_dz/2}"/>
-      <xacro:property name="arm_rpy" value="0 0 0"/>
-      <xacro:property name="extruder_xyz" value="0 0 ${extruder_h/2}"/>
-      <xacro:property name="extruder_rpy" value="0 0 ${-M_PI/2}"/>
-      <!-- includes -->
-      <xacro:include filename="$(find xarm_description)/urdf/xarm6_robot_macro.xacro" />
+      <xacro:property name="arm_xyz" value="${-0.185+base_link_dx/2} 0 ${0.005+0.028-base_link_dz/2}" />
+      <xacro:property name="arm_rpy" value="0 0 0" />
+      <xacro:property name="extruder_xyz" value="0 0 ${extruder_h/2}" />
+      <xacro:property name="extruder_rpy" value="0 0 ${-M_PI/2}" />
       <!-- formation-->
-      <xacro:include filename="$(find as_description)/robots/as_base.xacro" />
+      <xacro:as_base load_gazebo_plugin="$(arg load_gazebo_plugin)" />
       <xacro:xarm6_robot prefix="$(arg prefix)" namespace="$(arg ros_namespace)" limited="$(arg limited)" effort_control="$(arg effort_control)" velocity_control="$(arg velocity_control)" attach_to="base_link" xyz="${arm_xyz}" rpy="${arm_rpy}" load_gazebo_plugin="$(arg load_gazebo_plugin)" />
       <xacro:extruder parent="xarmlink_eef" xyz="${extruder_xyz}" rpy="${extruder_rpy}" />
+      <!-- Gazebo: My current understanding is that libgazebo_ros_control is a per-model-plugin
+      and most recent spawn will override the last one. So there is no nice way to namespace this.
+      Therefore the approach here disables individual base/arm plugins and launches a common one -->
+      <gazebo>
+            <plugin name="armstone_gazebo_ros_control" filename="libgazebo_ros_control.so">
+                  <robotNamespace>/as_control</robotNamespace>
+            </plugin>
+      </gazebo>
 </robot>

File: as_description/robots/as_base.xacro (robot description, xacro)
@@ -1,35 +1,5 @@
 <?xml version="1.0"?>
 <robot xmlns:sensor="http://playerstage.sourceforge.net/gazebo/xmlschema/#sensor" xmlns:controller="http://playerstage.sourceforge.net/gazebo/xmlschema/#controller" xmlns:interface="http://playerstage.sourceforge.net/gazebo/xmlschema/#interface" xmlns:xacro="http://ros.org/wiki/xacro" name="as_base">
-	<!-- Import macro params -->
-	<xacro:include filename="$(find as_description)/urdf/base/chasis.params.xacro" />
-	<xacro:include filename="$(find as_description)/urdf/base/components.params.xacro" />
-	<!-- Componenet positions-->
-	<xacro:property name="dc_box_xyz" value=" ${-base_link_dx/2 + 0.02 +dc_box_dy/2} 0 ${base_link_dz/2 - dc_box_dz/2}" />
-	<xacro:property name="dc_box_rpy" value=" 0 0 0" />
-	<xacro:property name="material3_xyz" value="-${base_link_dx/4} 0 ${base_link_dz/2+0.01 + battery_link_dz/2}" />
-	<xacro:property name="material3_rpy" value="0 ${M_PI/2} 0" />
-	<xacro:property name="mount_plate_xyz" value=" ${base_link_dx/2 - mount_plate_dx/2} 0 ${ -base_link_dz/2 +mount_plate_dz/2 +0.02}" />
-	<xacro:property name="mount_plate_rpy" value="0 0 0" />
-	<xacro:property name="compressor_xyz" value="-${base_link_dx/2-compressor_h/2 } ${base_link_dy/2 - compressor_r/2} ${base_link_dz/2-compressor_r }" />
-	<xacro:property name="compressor_rpy" value="0 ${M_PI/2} 0" />
-	<xacro:property name="battery_xyz" value="${-base_link_dx/2 + battery_link_dx/2 -0.08} 0  ${-base_link_dz/2 +0.02 + battery_link_dz/2 }" />
-	<xacro:property name="battery_rpy" value="0 0 0" />
-	<!-- Import macros -->
-	<xacro:include filename="$(find as_description)/urdf/base/chasis.macro.xacro" />
-	<xacro:include filename="$(find as_description)/urdf/base/components.macro.xacro" />
-	<!-- Compose the ArmStone Base -->
-	<xacro:as_base_chasis />
-	<xacro:battery48 parent="base_link" xyz="${battery_xyz}" rpy="${battery_rpy}" />
-	<xacro:dc_box parent="base_link" xyz="${dc_box_xyz}" rpy="${dc_box_rpy}" />
-	<xacro:mount_plate parent="base_link" xyz="${mount_plate_xyz}" rpy="${mount_plate_rpy}" />
-	<!-- <xacro:compressor parent="base_link" xyz="${compressor_xyz}" rpy="${compressor_rpy}" /> -->
-	<!-- <xacro:material3 parent="base_link" xyz="${material3_xyz}" rpy="${material3_rpy}" /> -->
-	<!-- gazebo_plugin -->
-	<!-- <xacro:if value="${load_gazebo_plugin}"> -->
-		<gazebo>
-			<plugin name="gazebo_ros_control" filename="libgazebo_ros_control.so">
-				<robotNamespace>/as_base</robotNamespace>
-			</plugin>
-		</gazebo>
-	<!-- </xacro:if> -->
+	<xacro:include filename="$(find as_description)/urdf/base/as_base.macro.xacro" />
+	<xacro:as_base />
 </robot>

File: as_description/urdf/base/chasis.macro.xacro (robot description, xacro)
@@ -7,5 +7,5 @@
 	<xacro:include filename="$(find as_description)/urdf/common/inertia.xacro"/>
 	<xacro:include filename="$(find as_description)/urdf/common/materials.xacro"/>
-	<xacro:macro name="as_motor_wheel_assembly" params="suffix wheel_angle  " >
+	<xacro:macro name="as_motor_wheel_assembly" params="suffix wheel_angle axis " >
 		<link name="motor_gearbox${suffix}">
 			<inertial>
@@ -30,5 +30,5 @@
 			<child link="omniwheel${suffix}"/>
 			<origin xyz= "0 0 ${motor_link_h/2}" rpy = "0 ${wheel_angle} 0" />
-			<axis xyz="0 0 1"/>
+			<axis xyz="${axis}"/>
 			<limit effort = "${motor_effort_limit}" velocity = "${motor_velocity_limit}" />
 			<dynamics damping="1.5" friction="1.0"/>
@@ -59,15 +59,20 @@
 				<!-- dummy visual so gazebo doesnt freakout -->
 				<geometry>
-					<sphere radius="${wheel_link_r/10}"/>
+					<sphere radius="${wheel_link_r/3}"/>
 				</geometry>
 			</visual>
+			<surface>
+				<bounce restitution_coefficient="0.0001" />
+			</surface>
 		</link>
 		<gazebo reference="omniwheel${suffix}">
-			<mu1 value="0.2"/>
+			<!-- not sure if mu or mu1 is used -->
+			<mu value="0.15"/>
+			<mu1 value="0.15"/>
 			<mu2 value="1.5"/>
 			<kp value="10000000.0" />
 			<kd value="10000.0" />
-			<fdir1 value="0 0 1"/>
-			<maxContacts value= "1"/>
+			<fdir1 value="1 0 0"/>
+			<!-- <maxContacts value= "1"/> -->
 			<material>Gazebo/White</material>
 		</gazebo>
@@ -110,8 +115,8 @@
 			</gazebo>
 		</link>
-		<xacro:as_motor_wheel_assembly suffix="_fl"  wheel_angle="${-wheel_roller_angle}"/>
-		<xacro:as_motor_wheel_assembly suffix="_fr"  wheel_angle="${wheel_roller_angle}"/>
-		<xacro:as_motor_wheel_assembly suffix="_bl"  wheel_angle="${wheel_roller_angle}"/>
-		<xacro:as_motor_wheel_assembly suffix="_br"  wheel_angle="${-wheel_roller_angle}"/>
+		<xacro:as_motor_wheel_assembly suffix="_fl"  wheel_angle="${wheel_roller_angle}" axis="-1 0 0"/>
+		<xacro:as_motor_wheel_assembly suffix="_fr"  wheel_angle="${-wheel_roller_angle}" axis="-1 0 0"/>
+		<xacro:as_motor_wheel_assembly suffix="_bl"  wheel_angle="${-wheel_roller_angle}" axis="1 0 0"/>
+		<xacro:as_motor_wheel_assembly suffix="_br"  wheel_angle="${wheel_roller_angle}" axis="1 0 0"/>
 		<joint name="motor_wheel_assembly_joint_fl" type="fixed">
 			<parent link="base_link"/>

File: as_description/urdf/base/chasis.params.xacro (robot description, xacro)
@@ -27,9 +27,14 @@
 	<xacro:property name="motor_mxyz" value="0 ${motor_link_r/2 +0.012} 0.025" />
 	<xacro:property name="motor_meshfile" value="motor.dae" />
-	<!-- True is 1460mNm -->
-	<xacro:property name="motor_effort_limit" value="50" />
-	<!-- True is 6110rpm. Which is 7.031 rad/s I think. So 5 to be safe.-->
+	<!-- with gearbox -->
+	<!-- True is 1460mNm  pre gearbox-->
+	<!-- True is 6110rpm. Which is 639 rad/s I think.-->
+	<!-- <xacro:property name="motor_effort_limit" value="1.4" />
+	<xacro:property name="motor_velocity_limit" value="600" />
+	<xacro:property name="gearbox_reduction" value="91" /> -->
+	<!-- Without gearbox sim -->
+	<!--safe values hopefulle  -->
+	<xacro:property name="motor_effort_limit" value="100" />
 	<xacro:property name="motor_velocity_limit" value="5" />
-	<!-- <xacro:property name="gearbox_reduction" value="91" /> -->
 	<xacro:property name="gearbox_reduction" value="1" />
 	<!-- offsets -->

Commit message: WIP

File: as_description/robots/as.xacro (robot description, xacro)
@@ -12,4 +12,5 @@
       <xacro:arg name="velocity_control" default="false" />
       <xacro:arg name="load_gazebo_plugin" default="false" />
+      <xacro:arg name="load_sensors" default="false" />
       <!-- placement -->
       <xacro:property name="arm_xyz" value="${-0.185+base_link_dx/2} 0 ${0.005+0.028-base_link_dz/2}" />
@@ -18,5 +19,5 @@
       <xacro:property name="extruder_rpy" value="0 0 ${-M_PI/2}" />
       <!-- formation-->
-      <xacro:as_base load_gazebo_plugin="$(arg load_gazebo_plugin)" />
+      <xacro:as_base load_gazebo_plugin="$(arg load_gazebo_plugin)" load_sensors="$(arg load_sensors)"/>
       <!-- explicit xarm_mount for easier robcogen -->
       <link name="xarm_mount">
@@ -28,5 +29,5 @@
       </joint>
       <xacro:xarm6_robot prefix="$(arg prefix)" namespace="$(arg ros_namespace)" limited="$(arg limited)" effort_control="$(arg effort_control)" velocity_control="$(arg velocity_control)" attach_to="xarm_mount" xyz="0 0 0" rpy="0 0 0" load_gazebo_plugin="$(arg load_gazebo_plugin)" />
-      <xacro:extruder parent="xarmlink_eef" xyz="${extruder_xyz}" rpy="${extruder_rpy}" />
+      <xacro:extruder parent="xarmlink_eef" xyz="${extruder_xyz}" rpy="${extruder_rpy}" load_sensors="$(arg load_sensors)"/>
       <!-- Gazebo: My current understanding is that libgazebo_ros_control is a per-model-plugin
       and most recent spawn will override the last one. So there is no nice way to namespace this.

File: as_description/urdf/base/as_base.macro.xacro (robot description, xacro)
@@ -31,5 +31,5 @@
 	<xacro:property name="right_hokuyo_xyz" value="${-base_link_dx/2 + 0.235} ${-base_link_dy/2  + 0.02 }  0" />
 	<xacro:property name="right_hokuyo_rpy" value="0 0 ${- M_PI/2}" />
-	<xacro:macro name="as_base" params="load_gazebo_plugin='true'">
+	<xacro:macro name="as_base" params="load_gazebo_plugin='true' load_sensors='true'">
 		<!-- Compose the ArmStone Base -->
 		<xacro:as_base_chasis />
@@ -44,8 +44,10 @@
 		<xacro:backpack parent="base_link" xyz="${backpack_xyz}" rpy="${backpack_rpy}" />
 		<!-- Sensors -->
-		<xacro:imu prefix="base" parent="base_link" xyz="${base_imu_xyz}" rpy="${base_imu_rpy}" />
-		<xacro:hokuyo prefix="left" parent="base_link" xyz="${left_hokuyo_xyz}" rpy="${left_hokuyo_rpy}" />
-		<xacro:hokuyo prefix="right" parent="base_link" xyz="${right_hokuyo_xyz}" rpy="${right_hokuyo_rpy}" />
-		<xacro:perfect_lidar parent="base_link" />
+		<xacro:if value="${load_sensors}">
+			<xacro:imu prefix="base" parent="base_link" xyz="${base_imu_xyz}" rpy="${base_imu_rpy}" />
+			<xacro:hokuyo prefix="left" parent="base_link" xyz="${left_hokuyo_xyz}" rpy="${left_hokuyo_rpy}" />
+			<xacro:hokuyo prefix="right" parent="base_link" xyz="${right_hokuyo_xyz}" rpy="${right_hokuyo_rpy}" />
+			<xacro:perfect_lidar parent="base_link" />
+		</xacro:if>
 	</xacro:macro>
 </robot>

File: as_description/urdf/base/components.macro.xacro (robot description, xacro)
@@ -61,5 +61,5 @@
 		<xacro:generic_box name="ic" parent="${parent}" xyz="${xyz}" rpy="${rpy}" dx="${ic_box_dx}" dy="${ic_box_dy}" dz="${ic_box_dz}" m="${ic_m}" material="LightGrey" gmaterial="Gazebo/LightGrey" meshfile="intermediate_assembly${mesh_filetype}" mxyz="${ic_box_dx/2 - 0.03} 0 ${-ic_box_dz/2}" mrpy="0 0 0" />
 	</xacro:macro>
-	<xacro:macro name="extruder" params="parent xyz rpy">
+	<xacro:macro name="extruder" params="parent xyz rpy load_sensors='true'">
 		<joint name="extruder_joint" type="fixed">
 			<parent link="${parent}" />
@@ -92,10 +92,12 @@
 		</joint>
 		<link name="extruder_ee" />
-		<xacro:imu prefix="ee" parent="${parent}" xyz="${ee_imu_xyz}" rpy="${ee_imu_rpy}" />
+		<xacro:if value="${load_sensors}">
+			<xacro:imu prefix="ee" parent="${parent}" xyz="${ee_imu_xyz}" rpy="${ee_imu_rpy}" />
+		</xacro:if>
 		<!-- Extruder Axes -->
 		<joint name="extruder_axes_joint" type="fixed">
 			<parent link="${parent}" />
 			<child link="extruder_axes_link" />
-			<origin xyz="0.018177 0.038884 -0.001" rpy="0 ${M_PI} ${-M_PI/2}" />
+			<origin xyz="0.018177 0.04388428 -0.001" rpy="0 ${M_PI} ${-M_PI/2}" />
 		</joint>
 		<link name="extruder_axes_link">
@@ -106,10 +108,10 @@
 				</geometry>
 			</visual>
-			<collision>
+			<!-- <collision>
 				<origin xyz="0 0 0" rpy="0 0 0" />
 				<geometry>
 					<mesh filename="package://as_description/meshes/extruder_axes${mesh_filetype}" />
 				</geometry>
-			</collision>
+			</collision> -->
 		</link>
 		<!-- LEFT is D435 -->
@@ -126,10 +128,10 @@
 				</geometry>
 			</visual>
-			<collision>
-				<origin xyz="0 0 0" rpy="0 0 0" />
-				<geometry>
-					<mesh filename="package://as_description/meshes/cam_holder${mesh_filetype}" />
-				</geometry>
-			</collision>
+			<!-- <collision>
+				<origin xyz="0 0 0" rpy="0 0 0" />
+				<geometry>
+					<mesh filename="package://as_description/meshes/cam_holder${mesh_filetype}" />
+				</geometry>
+			</collision> -->
 		</link>
 		<joint name="d435_mount_joint" type="fixed">
@@ -152,10 +154,10 @@
 				</geometry>
 			</visual>
-			<collision>
-				<origin xyz="0 0 0" rpy="0 0 0" />
-				<geometry>
-					<mesh filename="package://as_description/meshes/cam_holder${mesh_filetype}" />
-				</geometry>
-			</collision>
+			<!-- <collision>
+				<origin xyz="0 0 0" rpy="0 0 0" />
+				<geometry>
+					<mesh filename="package://as_description/meshes/cam_holder${mesh_filetype}" />
+				</geometry>
+			</collision> -->
 		</link>
 		<joint name="l515_mount_joint" type="fixed">
@@ -168,9 +170,11 @@
 		</joint>
 		<link name="l515_mount_link" />
-		<xacro:sensor_l515 name="l515_mount_link" topics_ns="/as_sensors/l515/depth_cam" parent="l515_mount_link" use_nominal_extrinsics="true" publish_pointcloud="true" add_plug="false" use_mesh="true">
+		<xacro:if value="${load_sensors}">
+			<xacro:sensor_l515 name="l515_mount_link" topics_ns="/as_sensors/l515/depth_cam" parent="l515_mount_link" use_nominal_extrinsics="true" publish_pointcloud="true" add_plug="false" use_mesh="true">
 			<origin xyz="0.01015 0  0.014" rpy="0 ${-M_PI/2} 0" />
 			<!-- From starting frame to screw hole closer to usb-c: -0.014;0;0.01015 -->
 			<!-- From starting frame to screw hole further to usb-c: -0.014;0;0.05015 -->
-		</xacro:sensor_l515>
+			</xacro:sensor_l515>
+		</xacro:if>
 		<!-- <xacro:sensor_d435 parent="d435_mount_link" use_nominal_extrinsics="true" add_plug="false" use_mesh="true">
 			<origin xyz="0 0 0" rpy="0 0 0"/>

Commit message: .

File: as_description/robots/as.xacro (robot description, xacro)
@@ -14,5 +14,5 @@
       <xacro:arg name="load_sensors" default="true" />
       <!-- placement -->
-      <xacro:property name="arm_xyz" value="${-0.185+base_link_dx/2} 0 ${0.005+0.028-base_link_dz/2}" />
+      <xacro:property name="arm_xyz" value="${-0.18500523+base_link_dx/2} 0 ${0.028-base_link_dz/2}" />
       <xacro:property name="arm_rpy" value="0 0 0" />
       <xacro:property name="extruder_xyz" value="0 0 ${extruder_h/2}" />
