Commit message: assembly typo

File: as_description/urdf/base/as_base.xacro (robot description, xacro)
@@ -38,12 +38,12 @@
 	<xacro:property name="nuc_link_m" value="0.3"/>
 	<!-- offsets -->
-	<xacro:property name="motor_wheel_assemply_xyz_fl" value="0.375 0.25 -0.08"/>
-	<xacro:property name="motor_wheel_assemply_rpy_fl" value="${- M_PI/2} 0 0"/>
-	<xacro:property name="motor_wheel_assemply_xyz_fr" value="0.375 -0.25 -0.08"/>
-	<xacro:property name="motor_wheel_assemply_rpy_fr" value="${M_PI/2} 0 0"/>
-	<xacro:property name="motor_wheel_assemply_xyz_bl" value="-0.375 0.25 -0.08"/>
-	<xacro:property name="motor_wheel_assemply_rpy_bl" value="${ M_PI/2} 0 ${M_PI}"/>
-	<xacro:property name="motor_wheel_assemply_xyz_br" value="-0.375 -0.25 -0.08"/>
-	<xacro:property name="motor_wheel_assemply_rpy_br" value="${-M_PI/2} 0 ${M_PI}"/>
+	<xacro:property name="motor_wheel_assembly_xyz_fl" value="0.375 0.25 -0.08"/>
+	<xacro:property name="motor_wheel_assembly_rpy_fl" value="${- M_PI/2} 0 0"/>
+	<xacro:property name="motor_wheel_assembly_xyz_fr" value="0.375 -0.25 -0.08"/>
+	<xacro:property name="motor_wheel_assembly_rpy_fr" value="${M_PI/2} 0 0"/>
+	<xacro:property name="motor_wheel_assembly_xyz_bl" value="-0.375 0.25 -0.08"/>
+	<xacro:property name="motor_wheel_assembly_rpy_bl" value="${ M_PI/2} 0 ${M_PI}"/>
+	<xacro:property name="motor_wheel_assembly_xyz_br" value="-0.375 -0.25 -0.08"/>
+	<xacro:property name="motor_wheel_assembly_rpy_br" value="${-M_PI/2} 0 ${M_PI}"/>
 	<xacro:property name="ground_clearance" value="0.05"/>
 	<xacro:macro name="as_motor_wheel_assembly" params="suffix">
@@ -155,20 +155,20 @@
 			<parent link="base_link"/>
 			<child link="motor_gearbox_fl"/>
-			<origin xyz= "${motor_wheel_assemply_xyz_fl}" rpy = "${motor_wheel_assemply_rpy_fl}" />
+			<origin xyz= "${motor_wheel_assembly_xyz_fl}" rpy = "${motor_wheel_assembly_rpy_fl}" />
 		</joint>
 		<joint name="motor_wheel_assembly_joint_fr" type="fixed">
 			<parent link="base_link"/>
 			<child link="motor_gearbox_fr"/>
-			<origin xyz= "${motor_wheel_assemply_xyz_fr}" rpy = "${motor_wheel_assemply_rpy_fr}" />
+			<origin xyz= "${motor_wheel_assembly_xyz_fr}" rpy = "${motor_wheel_assembly_rpy_fr}" />
 		</joint>
 		<joint name="motor_wheel_assembly_joint_bl" type="fixed">
 			<parent link="base_link"/>
 			<child link="motor_gearbox_bl"/>
-			<origin xyz= "${motor_wheel_assemply_xyz_bl}" rpy = "${motor_wheel_assemply_rpy_bl}" />
+			<origin xyz= "${motor_wheel_assembly_xyz_bl}" rpy = "${motor_wheel_assembly_rpy_bl}" />
 		</joint>
 		<joint name="motor_wheel_assembly_joint_br" type="fixed">
 			<parent link="base_link"/>
 			<child link="motor_gearbox_br"/>
-			<origin xyz= "${motor_wheel_assemply_xyz_br}" rpy = "${motor_wheel_assemply_rpy_br}" />
+			<origin xyz= "${motor_wheel_assembly_xyz_br}" rpy = "${motor_wheel_assembly_rpy_br}" />
 		</joint>
 		<gazebo>

File: as_description/urdf/base/asbase.xacro (robot description, xacro)
@@ -27,12 +27,12 @@
 	<xacro:property name="gearbox_reduction" value="91"/>
 	<!-- offsets -->
-	<xacro:property name="motor_wheel_assemply_xyz_fl" value="${base_link_dx/2-0.05} ${base_link_dy/2 -motor_link_h/2} -${base_link_dz/2 + motor_link_r/2}"/>
-	<xacro:property name="motor_wheel_assemply_rpy_fl" value="${- M_PI/2} 0 0"/>
-	<xacro:property name="motor_wheel_assemply_xyz_fr" value="${base_link_dx/2-0.05} -${base_link_dy/2 -motor_link_h/2} -${base_link_dz/2 + motor_link_r/2}"/>
-	<xacro:property name="motor_wheel_assemply_rpy_fr" value="${M_PI/2} 0 0"/>
-	<xacro:property name="motor_wheel_assemply_xyz_bl" value="-${base_link_dx/2-0.05} ${base_link_dy/2 -motor_link_h/2} -${base_link_dz/2 + motor_link_r/2}"/>
-	<xacro:property name="motor_wheel_assemply_rpy_bl" value="${ M_PI/2} 0 ${M_PI}"/>
-	<xacro:property name="motor_wheel_assemply_xyz_br" value="-${base_link_dx/2-0.05} -${base_link_dy/2 -motor_link_h/2} -${base_link_dz/2 + motor_link_r/2}"/>
-	<xacro:property name="motor_wheel_assemply_rpy_br" value="${-M_PI/2} 0 ${M_PI}"/>
+	<xacro:property name="motor_wheel_assembly_xyz_fl" value="${base_link_dx/2-0.05} ${base_link_dy/2 -motor_link_h/2} -${base_link_dz/2 + motor_link_r/2}"/>
+	<xacro:property name="motor_wheel_assembly_rpy_fl" value="${- M_PI/2} 0 0"/>
+	<xacro:property name="motor_wheel_assembly_xyz_fr" value="${base_link_dx/2-0.05} -${base_link_dy/2 -motor_link_h/2} -${base_link_dz/2 + motor_link_r/2}"/>
+	<xacro:property name="motor_wheel_assembly_rpy_fr" value="${M_PI/2} 0 0"/>
+	<xacro:property name="motor_wheel_assembly_xyz_bl" value="-${base_link_dx/2-0.05} ${base_link_dy/2 -motor_link_h/2} -${base_link_dz/2 + motor_link_r/2}"/>
+	<xacro:property name="motor_wheel_assembly_rpy_bl" value="${ M_PI/2} 0 ${M_PI}"/>
+	<xacro:property name="motor_wheel_assembly_xyz_br" value="-${base_link_dx/2-0.05} -${base_link_dy/2 -motor_link_h/2} -${base_link_dz/2 + motor_link_r/2}"/>
+	<xacro:property name="motor_wheel_assembly_rpy_br" value="${-M_PI/2} 0 ${M_PI}"/>
 	<xacro:property name="ground_clearance" value="${motor_link_r/2 +wheel_link_r/2}"/>
 	<!-- Import Things -->

File: as_description/urdf/base/chasis.xacro (robot description, xacro)
@@ -115,20 +115,20 @@
 			<parent link="base_link"/>
 			<child link="motor_gearbox_fl"/>
-			<origin xyz= "${motor_wheel_assemply_xyz_fl}" rpy = "${motor_wheel_assemply_rpy_fl}" />
+			<origin xyz= "${motor_wheel_assembly_xyz_fl}" rpy = "${motor_wheel_assembly_rpy_fl}" />
 		</joint>
 		<joint name="motor_wheel_assembly_joint_fr" type="fixed">
 			<parent link="base_link"/>
 			<child link="motor_gearbox_fr"/>
-			<origin xyz= "${motor_wheel_assemply_xyz_fr}" rpy = "${motor_wheel_assemply_rpy_fr}" />
+			<origin xyz= "${motor_wheel_assembly_xyz_fr}" rpy = "${motor_wheel_assembly_rpy_fr}" />
 		</joint>
 		<joint name="motor_wheel_assembly_joint_bl" type="fixed">
 			<parent link="base_link"/>
 			<child link="motor_gearbox_bl"/>
-			<origin xyz= "${motor_wheel_assemply_xyz_bl}" rpy = "${motor_wheel_assemply_rpy_bl}" />
+			<origin xyz= "${motor_wheel_assembly_xyz_bl}" rpy = "${motor_wheel_assembly_rpy_bl}" />
 		</joint>
 		<joint name="motor_wheel_assembly_joint_br" type="fixed">
 			<parent link="base_link"/>
 			<child link="motor_gearbox_br"/>
-			<origin xyz= "${motor_wheel_assemply_xyz_br}" rpy = "${motor_wheel_assemply_rpy_br}" />
+			<origin xyz= "${motor_wheel_assembly_xyz_br}" rpy = "${motor_wheel_assembly_rpy_br}" />
 		</joint>
 		<gazebo>
