Commit message: Sunday nigth joystick

File: as_description/urdf/base/chasis.params.xacro (robot description, xacro)
@@ -24,5 +24,5 @@
 	<xacro:property name="motor_effort_limit" value="1.4" />
 	<!-- True is 6110rpm -->
-	<xacro:property name="motor_velocity_limit" value="600" />
+	<xacro:property name="motor_velocity_limit" value="8" />
 	<xacro:property name="gearbox_reduction" value="91" />
 	<!-- offsets -->

Commit message: Change description joint limits

File: as_description/urdf/base/chasis.params.xacro (robot description, xacro)
@@ -22,7 +22,7 @@
 	<xacro:property name="motor_link_m" value="${0.14 +0.36}" />
 	<!-- True is 1460mNm -->
-	<xacro:property name="motor_effort_limit" value="1.4" />
+	<xacro:property name="motor_effort_limit" value="1" />
 	<!-- True is 6110rpm -->
-	<xacro:property name="motor_velocity_limit" value="8" />
+	<xacro:property name="motor_velocity_limit" value="4" />
 	<xacro:property name="gearbox_reduction" value="91" />
 	<!-- offsets -->

Commit message: mecanum stack WIP

File: as_description/urdf/base/chasis.params.xacro (robot description, xacro)
@@ -24,5 +24,5 @@
 	<xacro:property name="motor_effort_limit" value="1" />
 	<!-- True is 6110rpm -->
-	<xacro:property name="motor_velocity_limit" value="6" />
+	<xacro:property name="motor_velocity_limit" value="5" />
 	<xacro:property name="gearbox_reduction" value="91" />
 	<!-- offsets -->
