Commit message: FIxes to description architecture

File: as_description/urdf/base/chasis.macro.xacro (robot description, xacro)
@@ -7,44 +7,4 @@
 	<xacro:include filename="$(find as_description)/urdf/common/inertia.xacro"/>
 	<xacro:include filename="$(find as_description)/urdf/common/materials.xacro"/>
-	<!-- Link Dimensions -->
-	<!-- base_link -->
-	<xacro:property name="base_link_dx" value="0.8"/>
-	<xacro:property name="base_link_dy" value="0.5"/>
-	<xacro:property name="base_link_dz" value="0.2"/>
-	<xacro:property name="base_link_m" value="2"/>
-	<!-- alluminium frame only -->
-	<!-- wheel_link -->
-	<xacro:property name="wheel_link_r" value="${0.152/2}"/>
-	<xacro:property name="wheel_link_m" value="0.6"/>
-	<xacro:property name="wheel_roller_angle" value="${45*M_PI/180}"/>
-	<!-- motor_gearbox_link -->
-	<xacro:property name="motor_link_r" value="0.025"/>
-	<xacro:property name="motor_link_h" value="0.12"/>
-	<xacro:property name="motor_link_m" value="0.5"/>
-	<!-- True is 1460mNm -->
-	<xacro:property name="motor_effort_limit" value="1.4"/>
-	<!-- True is 6110rpm -->
-	<xacro:property name="motor_velocity_limit" value="600"/>
-	<xacro:property name="gearbox_reduction" value="91"/>
-	<!-- battery_link -->
-	<xacro:property name="battery_link_dx" value="0.8"/>
-	<xacro:property name="battery_link_dy" value="0.5"/>
-	<xacro:property name="battery_link_dz" value="0.2"/>
-	<xacro:property name="battery_link_m" value="6.7"/>
-	<!-- nuc_link -->
-	<xacro:property name="nuc_link_dx" value="0.12"/>
-	<xacro:property name="nuc_link_dy" value="0.12"/>
-	<xacro:property name="nuc_link_dz" value="0.06"/>
-	<xacro:property name="nuc_link_m" value="0.3"/>
-	<!-- offsets -->
-	<xacro:property name="motor_wheel_assembly_xyz_fl" value="0.375 0.25 -0.08"/>
-	<xacro:property name="motor_wheel_assembly_rpy_fl" value="${- M_PI/2} 0 0"/>
-	<xacro:property name="motor_wheel_assembly_xyz_fr" value="0.375 -0.25 -0.08"/>
-	<xacro:property name="motor_wheel_assembly_rpy_fr" value="${M_PI/2} 0 0"/>
-	<xacro:property name="motor_wheel_assembly_xyz_bl" value="-0.375 0.25 -0.08"/>
-	<xacro:property name="motor_wheel_assembly_rpy_bl" value="${ M_PI/2} 0 ${M_PI}"/>
-	<xacro:property name="motor_wheel_assembly_xyz_br" value="-0.375 -0.25 -0.08"/>
-	<xacro:property name="motor_wheel_assembly_rpy_br" value="${-M_PI/2} 0 ${M_PI}"/>
-	<xacro:property name="ground_clearance" value="0.05"/>
 	<xacro:macro name="as_motor_wheel_assembly" params="suffix">
 		<link name="motor_gearbox${suffix}">
@@ -111,5 +71,5 @@
 		</gazebo>
 	</xacro:macro>
-	<xacro:macro name="as_base">
+	<xacro:macro name="as_base_chasis">
 		<!-- Projection of base_link origin to xy plane -->
 		<link name="base_link_footprint"/>
@@ -174,5 +134,5 @@
 		<gazebo>
 			<plugin name="gazebo_ros_control" filename="libgazebo_ros_control.so">
-				<robotNamespace>/asbase</robotNamespace>
+				<robotNamespace>/as_base</robotNamespace>
 			</plugin>
 		</gazebo>

Commit message: control stack debugged with diff drive controller

File: as_description/urdf/base/chasis.macro.xacro (robot description, xacro)
@@ -32,5 +32,5 @@
 			<axis xyz="0 0 1"/>
 			<limit effort = "${motor_effort_limit}" velocity = "${motor_velocity_limit}" />
-			<dynamics damping="1.5"/>
+			<!-- <dynamics damping="1.5"/> -->
 		</joint>
 		<transmission name="motor_wheel_joint_transmission${suffix}">

File: as_description/urdf/base/chasis.params.xacro (robot description, xacro)
@@ -24,5 +24,5 @@
 	<xacro:property name="motor_effort_limit" value="1" />
 	<!-- True is 6110rpm -->
-	<xacro:property name="motor_velocity_limit" value="4" />
+	<xacro:property name="motor_velocity_limit" value="6" />
 	<xacro:property name="gearbox_reduction" value="91" />
 	<!-- offsets -->

Commit message: Fixed gazebo spawn and added better extruder collisionbox

File: as_description/urdf/base/chasis.macro.xacro (robot description, xacro)
@@ -56,4 +56,10 @@
 				</geometry>
 			</collision>
+			<visual>
+				<!-- dummy visual so gazebo doesnt freakout -->
+				<geometry>
+					<sphere radius="${wheel_link_r/10}"/>
+				</geometry>
+			</visual>
 		</link>
 		<gazebo reference="omniwheel${suffix}">

File: as_description/urdf/base/components.macro.xacro (robot description, xacro)
@@ -73,21 +73,12 @@
 					<mesh filename="package://as_description/meshes/extruder.dae" />
 				</geometry>
-                <material name="Red"/>
             </visual>
             <collision>
-                <geometry>
-                    <cylinder radius="${extruder_r}" length="${extruder_h}" />
-                </geometry>
-            </collision>
-			<collision>
-				<origin xyz= "0 0 ${-extruder_h/2}" rpy = "0 0 0" />
-                <geometry>
-                    <cylinder radius="${extruder_r*1.5}" length="${extruder_h/2}" />
-                </geometry>
+                <origin xyz= "0 0 ${-extruder_h/2}" rpy = "0 0 0" />
+				<geometry>
+					<mesh filename="package://as_description/meshes/extruder_collision.dae" />
+				</geometry>
             </collision>
         </link>
-		<gazebo reference="extruder_link">
-            <material>Gazebo/Red</material>
-        </gazebo>
 		<link name="extruder_ee"/>
 		<joint name="extruder_ee_joint" type="fixed">

Commit message: see previous

File: as_description/urdf/base/chasis.macro.xacro (robot description, xacro)
@@ -1,19 +1,16 @@
 <?xml version="1.0"?>
-<robot xmlns:sensor="http://playerstage.sourceforge.net/gazebo/xmlschema/#sensor"
-	xmlns:controller="http://playerstage.sourceforge.net/gazebo/xmlschema/#controller"
-	xmlns:interface="http://playerstage.sourceforge.net/gazebo/xmlschema/#interface"
-	xmlns:xacro="http://ros.org/wiki/xacro">
+<robot xmlns:sensor="http://playerstage.sourceforge.net/gazebo/xmlschema/#sensor" xmlns:controller="http://playerstage.sourceforge.net/gazebo/xmlschema/#controller" xmlns:interface="http://playerstage.sourceforge.net/gazebo/xmlschema/#interface" xmlns:xacro="http://ros.org/wiki/xacro">
 	<!-- Common -->
-	<xacro:include filename="$(find as_description)/urdf/common/inertia.xacro"/>
-	<xacro:include filename="$(find as_description)/urdf/common/materials.xacro"/>
-	<xacro:macro name="as_motor_wheel_assembly" params="suffix wheel_angle axis " >
+	<xacro:include filename="$(find as_description)/urdf/common/inertia.xacro" />
+	<xacro:include filename="$(find as_description)/urdf/common/materials.xacro" />
+	<xacro:macro name="as_motor_wheel_assembly" params="suffix wheel_angle axis ">
 		<link name="motor_gearbox${suffix}">
 			<inertial>
-				<origin xyz="0 0 0" rpy="0 0 0"/>
-				<mass value="${motor_link_m}"/>
+				<origin xyz="0 0 0" rpy="0 0 0" />
+				<mass value="${motor_link_m}" />
 				<xacro:cylinder_inertia_tensor m="${motor_link_m}" r="${motor_link_r}" h="${motor_link_h}" />
 			</inertial>
 			<visual>
-				<origin xyz= "${motor_mxyz}" rpy = "${motor_mrpy}" />
+				<origin xyz="${motor_mxyz}" rpy="${motor_mrpy}" />
 				<geometry>
 					<mesh filename="package://as_description/meshes/${motor_meshfile}" />
@@ -22,15 +19,15 @@
 			<collision>
 				<geometry>
-					<cylinder length="${motor_link_h}" radius="${motor_link_r}"/>
+					<cylinder length="${motor_link_h}" radius="${motor_link_r}" />
 				</geometry>
 			</collision>
 		</link>
 		<joint name="motor_wheel_joint${suffix}" type="continuous">
-			<parent link="motor_gearbox${suffix}"/>
-			<child link="omniwheel${suffix}"/>
-			<origin xyz= "0 0 ${motor_link_h/2}" rpy = "0 ${wheel_angle} 0" />
-			<axis xyz="${axis}"/>
-			<limit effort = "${motor_effort_limit}" velocity = "${motor_velocity_limit}" />
-			<dynamics damping="1.5" friction="1.0"/>
+			<parent link="motor_gearbox${suffix}" />
+			<child link="omniwheel${suffix}" />
+			<origin xyz="0 0 ${motor_link_h/2}" rpy="0 ${wheel_angle} 0" />
+			<axis xyz="${axis}" />
+			<limit effort="${motor_effort_limit}" velocity="${motor_velocity_limit}" />
+			<dynamics damping="1.5" friction="1.0" />
 		</joint>
 		<transmission name="motor_wheel_joint_transmission${suffix}">
@@ -46,6 +43,6 @@
 		<link name="omniwheel${suffix}">
 			<inertial>
-				<origin xyz="0 0 0" rpy="0 0 0"/>
-				<mass value="${wheel_link_m}"/>
+				<origin xyz="0 0 0" rpy="0 0 0" />
+				<mass value="${wheel_link_m}" />
 				<xacro:sphere_inertia_tensor m="${wheel_link_m}" r="${wheel_link_r/2}" />
 			</inertial>
@@ -53,5 +50,5 @@
 			<collision>
 				<geometry>
-					<sphere radius="${wheel_link_r}"/>
+					<sphere radius="${wheel_link_r}" />
 				</geometry>
 			</collision>
@@ -59,5 +56,5 @@
 				<!-- dummy visual so gazebo doesnt freakout -->
 				<geometry>
-					<sphere radius="${wheel_link_r/3}"/>
+					<sphere radius="${wheel_link_r/3}" />
 				</geometry>
 			</visual>
@@ -68,9 +65,9 @@
 		<gazebo reference="omniwheel${suffix}">
 			<!-- not sure if mu or mu1 is used -->
-			<mu1 value="0.15"/>
-			<mu2 value="1.5"/>
+			<mu1 value="0.15" />
+			<mu2 value="1.5" />
 			<kp value="10000000.0" />
 			<kd value="10000.0" />
-			<fdir1 value="1 0 0"/>
+			<fdir1 value="1 0 0" />
 			<!-- <maxContacts value= "1"/> -->
 			<material>Gazebo/White</material>
@@ -79,26 +76,26 @@
 	<xacro:macro name="as_base_chasis">
 		<!-- Projection of base_link origin to xy plane -->
-		<link name="base_link_footprint"/>
+		<link name="base_link_footprint" />
 		<joint name="joint0" type="fixed">
-			<parent link="base_link_footprint"/>
-			<child link="base_link_base"/>
-			<origin xyz= "0 0 ${ground_clearance}" rpy = "0 0 0" />
+			<parent link="base_link_footprint" />
+			<child link="base_link_base" />
+			<origin xyz="0 0 ${ground_clearance}" rpy="0 0 0" />
 		</joint>
 		<!-- Projection of base_link origin to bottom of baselink collision box (i.e. raised only by wheels) -->
-		<link name="base_link_base"/>
+		<link name="base_link_base" />
 		<joint name="joint1" type="fixed">
-			<parent link="base_link_base"/>
-			<child link="base_link"/>
-			<origin xyz= "0 0 ${base_link_dz/2}" rpy = "0 0 0" />
+			<parent link="base_link_base" />
+			<child link="base_link" />
+			<origin xyz="0 0 ${base_link_dz/2}" rpy="0 0 0" />
 		</joint>
 		<!-- baselink -->
 		<link name="base_link">
 			<inertial>
-				<origin xyz="0 0 0" rpy="0 0 0"/>
-				<mass value="${base_link_m}"/>
-				<xacro:box_inertia_tensor m="${base_link_m}" dx="${base_link_dx}" dy="${base_link_dy}" dz="${base_link_dz}"/>
+				<origin xyz="0 0 0" rpy="0 0 0" />
+				<mass value="${base_link_m}" />
+				<xacro:box_inertia_tensor m="${base_link_m}" dx="${base_link_dx}" dy="${base_link_dy}" dz="${base_link_dz}" />
 			</inertial>
 			<visual>
-				<origin xyz= "${base_mxyz}" rpy = "${base_mrpy}" />
+				<origin xyz="${base_mxyz}" rpy="${base_mrpy}" />
 				<geometry>
 					<mesh filename="package://as_description/meshes/${base_meshfile}" />
@@ -106,5 +103,5 @@
 			</visual>
 			<collision>
-				<origin xyz= "-0.125 0 0" rpy = "0 0 0" />
+				<origin xyz="-0.125 0 0" rpy="0 0 0" />
 				<geometry>
 					<box size="${base_link_dx-0.25} ${base_link_dy} ${base_link_dz}" />
@@ -112,5 +109,5 @@
 			</collision>
 			<collision>
-				<origin xyz= "0 0 ${-(base_link_dz-0.03)/2}" rpy = "0 0 0" />
+				<origin xyz="0 0 ${-(base_link_dz-0.03)/2}" rpy="0 0 0" />
 				<geometry>
 					<box size="${base_link_dx} ${base_link_dy} 0.035" />
@@ -118,5 +115,5 @@
 			</collision>
 			<collision>
-				<origin xyz= "${base_link_dx/2 -0.125} ${base_link_dy/2 -0.01} 0.015" rpy = "0 ${-60*M_PI/180} 0" />
+				<origin xyz="${base_link_dx/2 -0.125} ${base_link_dy/2 -0.01} 0.015" rpy="0 ${-60*M_PI/180} 0" />
 				<geometry>
 					<box size=" 0.025 0.025 0.29" />
@@ -124,5 +121,5 @@
 			</collision>
 			<collision>
-				<origin xyz= "${base_link_dx/2 -0.125} ${-base_link_dy/2 +0.01} 0.015" rpy = "0 ${-60*M_PI/180} 0" />
+				<origin xyz="${base_link_dx/2 -0.125} ${-base_link_dy/2 +0.01} 0.015" rpy="0 ${-60*M_PI/180} 0" />
 				<geometry>
 					<box size=" 0.025 0.025 0.29" />
@@ -133,27 +130,27 @@
 			</gazebo>
 		</link>
-		<xacro:as_motor_wheel_assembly suffix="_fl"  wheel_angle="${wheel_roller_angle}" axis="-1 0 0"/>
-		<xacro:as_motor_wheel_assembly suffix="_fr"  wheel_angle="${-wheel_roller_angle}" axis="-1 0 0"/>
-		<xacro:as_motor_wheel_assembly suffix="_bl"  wheel_angle="${-wheel_roller_angle}" axis="1 0 0"/>
-		<xacro:as_motor_wheel_assembly suffix="_br"  wheel_angle="${wheel_roller_angle}" axis="1 0 0"/>
+		<xacro:as_motor_wheel_assembly suffix="_fl" wheel_angle="${wheel_roller_angle}" axis="-1 0 0" />
+		<xacro:as_motor_wheel_assembly suffix="_fr" wheel_angle="${-wheel_roller_angle}" axis="-1 0 0" />
+		<xacro:as_motor_wheel_assembly suffix="_bl" wheel_angle="${-wheel_roller_angle}" axis="1 0 0" />
+		<xacro:as_motor_wheel_assembly suffix="_br" wheel_angle="${wheel_roller_angle}" axis="1 0 0" />
 		<joint name="motor_wheel_assembly_joint_fl" type="fixed">
-			<parent link="base_link"/>
-			<child link="motor_gearbox_fl"/>
-			<origin xyz= "${motor_wheel_assembly_xyz_fl}" rpy = "${motor_wheel_assembly_rpy_fl}" />
+			<parent link="base_link" />
+			<child link="motor_gearbox_fl" />
+			<origin xyz="${motor_wheel_assembly_xyz_fl}" rpy="${motor_wheel_assembly_rpy_fl}" />
 		</joint>
 		<joint name="motor_wheel_assembly_joint_fr" type="fixed">
-			<parent link="base_link"/>
-			<child link="motor_gearbox_fr"/>
-			<origin xyz= "${motor_wheel_assembly_xyz_fr}" rpy = "${motor_wheel_assembly_rpy_fr}" />
+			<parent link="base_link" />
+			<child link="motor_gearbox_fr" />
+			<origin xyz="${motor_wheel_assembly_xyz_fr}" rpy="${motor_wheel_assembly_rpy_fr}" />
 		</joint>
 		<joint name="motor_wheel_assembly_joint_bl" type="fixed">
-			<parent link="base_link"/>
-			<child link="motor_gearbox_bl"/>
-			<origin xyz= "${motor_wheel_assembly_xyz_bl}" rpy = "${motor_wheel_assembly_rpy_bl}" />
+			<parent link="base_link" />
+			<child link="motor_gearbox_bl" />
+			<origin xyz="${motor_wheel_assembly_xyz_bl}" rpy="${motor_wheel_assembly_rpy_bl}" />
 		</joint>
 		<joint name="motor_wheel_assembly_joint_br" type="fixed">
-			<parent link="base_link"/>
-			<child link="motor_gearbox_br"/>
-			<origin xyz= "${motor_wheel_assembly_xyz_br}" rpy = "${motor_wheel_assembly_rpy_br}" />
+			<parent link="base_link" />
+			<child link="motor_gearbox_br" />
+			<origin xyz="${motor_wheel_assembly_xyz_br}" rpy="${motor_wheel_assembly_rpy_br}" />
 		</joint>
 	</xacro:macro>

File: as_description/urdf/base/chasis.params.xacro (robot description, xacro)
@@ -4,4 +4,6 @@
 	xmlns:interface="http://playerstage.sourceforge.net/gazebo/xmlschema/#interface"
 	xmlns:xacro="http://ros.org/wiki/xacro">
+	<xacro:property name="mesh_filetype" value=".dae" />
+	<!-- <xacro:property name="mesh_filetype" value=".stl" /> -->
 	<!-- Link Dimensions -->
 	<!-- base_link -->
@@ -11,5 +13,5 @@
 	<!-- 2.8kg raw frame. 3.5 estimate  full -->
 	<xacro:property name="base_link_m" value="3.5" />
-	<xacro:property name="base_meshfile" value="chasis.dae" />
+	<xacro:property name="base_meshfile" value="chasis${mesh_filetype}" />
 	<xacro:property name="base_mxyz" value="${(base_link_dx/2 - 0.01)} 0 ${(0.02 - 0.006 -base_link_dz/2)}" />
 	<xacro:property name="base_mrpy" value="0 0 0" />
@@ -26,5 +28,5 @@
 	<xacro:property name="motor_mrpy" value="${M_PI/2} ${- M_PI/2} 0" />
 	<xacro:property name="motor_mxyz" value="0 ${motor_link_r/2 +0.012} 0.025" />
-	<xacro:property name="motor_meshfile" value="motor.dae" />
+	<xacro:property name="motor_meshfile" value="motor${mesh_filetype}" />
 	<!-- with gearbox -->
 	<!-- True is 1460mNm  pre gearbox-->

File: as_description/urdf/base/components.macro.xacro (robot description, xacro)
@@ -3,4 +3,6 @@
 	<xacro:include filename="$(find as_description)/urdf/common/generic_links.xacro"/>
 	<xacro:include filename="$(find sensor_imu)/urdf/sensor_imu.xacro"/>
+	<xacro:property name="mesh_filetype" value=".dae" />
+	<!-- <xacro:property name="mesh_filetype" value=".stl" /> -->
 	<!-- battery_link -->
 	<xacro:property name="battery_link_dx" value="0.40"/>
@@ -38,5 +40,5 @@
 	<xacro:property name="ee_imu_rpy" value="0 3.14159265359 0"/>
 	<xacro:macro name="battery48" params="parent xyz rpy">
-		<xacro:generic_box name="battery48" parent="${parent}" xyz="${xyz}" rpy="${rpy}" dx="${battery_link_dx}" dy="${battery_link_dy}" dz="${battery_link_dz}" m="${battery_link_m}" material="LightGrey" gmaterial="Gazebo/LightGrey" meshfile="battery.dae" mxyz="0.035 0 ${-battery_link_dz/2}" mrpy="0 0 ${M_PI}" />
+		<xacro:generic_box name="battery48" parent="${parent}" xyz="${xyz}" rpy="${rpy}" dx="${battery_link_dx}" dy="${battery_link_dy}" dz="${battery_link_dz}" m="${battery_link_m}" material="LightGrey" gmaterial="Gazebo/LightGrey" meshfile="battery${mesh_filetype}" mxyz="0.035 0 ${-battery_link_dz/2}" mrpy="0 0 ${M_PI}" />
 	</xacro:macro>
 	<xacro:macro name="nuc" params="parent xyz rpy suffix">
@@ -44,5 +46,5 @@
 	</xacro:macro>
 	<xacro:macro name="dc_box" params="parent xyz rpy">
-		<xacro:generic_box name="dc_box" parent="${parent}" xyz="${xyz}" rpy="${rpy}" dx="${dc_box_dx}" dy="${dc_box_dy}" dz="${dc_box_dz}" m="${dc_box_m}" material="LightGrey" gmaterial="Gazebo/LightGrey" meshfile="dcbox.dae" mxyz="0 0 ${dc_box_dz/2}" mrpy="0 0 ${M_PI/2} " />
+		<xacro:generic_box name="dc_box" parent="${parent}" xyz="${xyz}" rpy="${rpy}" dx="${dc_box_dx}" dy="${dc_box_dy}" dz="${dc_box_dz}" m="${dc_box_m}" material="LightGrey" gmaterial="Gazebo/LightGrey" meshfile="dcbox${mesh_filetype}" mxyz="0 0 ${dc_box_dz/2}" mrpy="0 0 ${M_PI/2} " />
 	</xacro:macro>
 	<xacro:macro name="mount_plate" params="parent xyz rpy">
@@ -50,14 +52,14 @@
 	</xacro:macro>
 	<xacro:macro name="compressor" params="parent xyz rpy">
-		<xacro:generic_box name="compressor" parent="${parent}" xyz="${xyz}" rpy="${rpy}" dx="${compressor_box_dx}" dy="${compressor_box_dy}" dz="${compressor_box_dz}" m="${compressor_m}" material="Grey" gmaterial="Gazebo/Grey" meshfile="compressor_assembly.dae" mxyz="0 0 ${-compressor_box_dz/2}" mrpy="0 0 0" />
+		<xacro:generic_box name="compressor" parent="${parent}" xyz="${xyz}" rpy="${rpy}" dx="${compressor_box_dx}" dy="${compressor_box_dy}" dz="${compressor_box_dz}" m="${compressor_m}" material="Grey" gmaterial="Gazebo/Grey" meshfile="compressor_assembly${mesh_filetype}" mxyz="0 0 ${-compressor_box_dz/2}" mrpy="0 0 0" />
 	</xacro:macro>
 	<xacro:macro name="material3" params="parent xyz rpy">
-		<xacro:generic_cylinder name="material3" parent="${parent}" xyz="${xyz}" rpy="${rpy}" r="${material3_r}" h="${material3_h}" m="${material3_m}" material="LightGrey" gmaterial="Gazebo/LightGrey" meshfile="clay_assembly.dae" mxyz="${material3_r+0.02}  0  ${material3_h/5}" mrpy="0 ${-M_PI/2} 0"/>
+		<xacro:generic_cylinder name="material3" parent="${parent}" xyz="${xyz}" rpy="${rpy}" r="${material3_r}" h="${material3_h}" m="${material3_m}" material="LightGrey" gmaterial="Gazebo/LightGrey" meshfile="clay_assembly${mesh_filetype}" mxyz="${material3_r+0.02}  0  ${material3_h/5}" mrpy="0 ${-M_PI/2} 0"/>
 	</xacro:macro>
 	<xacro:macro name="cover_plate" params="parent xyz rpy">
-		<xacro:generic_box name="cover_plate" parent="${parent}" xyz="${xyz}" rpy="${rpy}" dx="${cover_box_dx}" dy="${cover_box_dy}" dz="${cover_box_dz}" m="${cover_plate_m}" material="LightGrey" gmaterial="Gazebo/LightGrey" meshfile="cover_assembly_.dae" mxyz="0 0 0" mrpy="0 0 0"/>
+		<xacro:generic_box name="cover_plate" parent="${parent}" xyz="${xyz}" rpy="${rpy}" dx="${cover_box_dx}" dy="${cover_box_dy}" dz="${cover_box_dz}" m="${cover_plate_m}" material="LightGrey" gmaterial="Gazebo/LightGrey" meshfile="cover_assembly_${mesh_filetype}" mxyz="0 0 0" mrpy="0 0 0"/>
 	</xacro:macro>
 	<xacro:macro name="ic" params="parent xyz rpy">
-		<xacro:generic_box name="ic" parent="${parent}" xyz="${xyz}" rpy="${rpy}" dx="${ic_box_dx}" dy="${ic_box_dy}" dz="${ic_box_dz}" m="${ic_m}" material="LightGrey" gmaterial="Gazebo/LightGrey" meshfile="intermediate_assembly.dae" mxyz="${ic_box_dx/2 - 0.03} 0 ${-ic_box_dz/2}" mrpy="0 0 0"/>
+		<xacro:generic_box name="ic" parent="${parent}" xyz="${xyz}" rpy="${rpy}" dx="${ic_box_dx}" dy="${ic_box_dy}" dz="${ic_box_dz}" m="${ic_m}" material="LightGrey" gmaterial="Gazebo/LightGrey" meshfile="intermediate_assembly${mesh_filetype}" mxyz="${ic_box_dx/2 - 0.03} 0 ${-ic_box_dz/2}" mrpy="0 0 0"/>
 	</xacro:macro>
 	<xacro:macro name="extruder" params="parent xyz rpy">
@@ -76,5 +78,5 @@
 				<origin xyz= "0 0 ${-extruder_h/2}" rpy = "0 0 0" />
 				<geometry>
-					<mesh filename="package://as_description/meshes/extruder.dae" />
+					<mesh filename="package://as_description/meshes/extruder${mesh_filetype}" />
 				</geometry>
             </visual>
@@ -82,5 +84,5 @@
                 <origin xyz= "0 0 ${-extruder_h/2}" rpy = "0 0 0" />
 				<geometry>
-					<mesh filename="package://as_description/meshes/extruder_collision.dae" />
+					<mesh filename="package://as_description/meshes/extruder_collision${mesh_filetype}" />
 				</geometry>
             </collision>
