Commit message: integrated imu sensors base and ee

File: as_description/urdf/base/as_base.macro.xacro (robot description, xacro)
@@ -7,4 +7,5 @@
 	<xacro:include filename="$(find as_description)/urdf/base/chasis.macro.xacro" />
 	<xacro:include filename="$(find as_description)/urdf/base/components.macro.xacro" />
+	<xacro:include filename="$(find sensor_imu)/urdf/sensor_imu.xacro" />
 	<!-- Componenet positions-->
 	<xacro:property name="dc_box_xyz" value=" ${-base_link_dx/2 + 0.02 +dc_box_dy/2} 0 ${base_link_dz/2 - dc_box_dz/2}" />
@@ -18,4 +19,6 @@
 	<xacro:property name="battery_xyz" value="${-base_link_dx/2 + battery_link_dx/2 -0.08} 0  ${-base_link_dz/2 +0.02 + battery_link_dz/2 }" />
 	<xacro:property name="battery_rpy" value="0 0 0" />
+	<xacro:property name="base_imu_xyz" value="${0.245 +(0.205/2)-(base_link_dx/2)} 0  ${-0.02+base_link_dz/2}" />
+	<xacro:property name="base_imu_rpy" value="0 0 0" />
 	<xacro:macro name="as_base" params="load_gazebo_plugin='true'">
 		<!-- Compose the ArmStone Base -->
@@ -24,4 +27,5 @@
 		<xacro:dc_box parent="base_link" xyz="${dc_box_xyz}" rpy="${dc_box_rpy}" />
 		<xacro:mount_plate parent="base_link" xyz="${mount_plate_xyz}" rpy="${mount_plate_rpy}" />
+		<xacro:imu prefix="base" parent="base_link" xyz="${base_imu_xyz}" rpy="${base_imu_rpy}" />
 		<!-- <xacro:compressor parent="base_link" xyz="${compressor_xyz}" rpy="${compressor_rpy}" /> -->
 		<!-- <xacro:material3 parent="base_link" xyz="${material3_xyz}" rpy="${material3_rpy}" /> -->

File: as_description/urdf/base/components.macro.xacro (robot description, xacro)
@@ -2,4 +2,5 @@
 <robot xmlns:xacro="http://ros.org/wiki/xacro">
 	<xacro:include filename="$(find as_description)/urdf/common/generic_links.xacro"/>
+	<xacro:include filename="$(find sensor_imu)/urdf/sensor_imu.xacro"/>
 	<!-- battery_link -->
 	<xacro:property name="battery_link_dx" value="0.40"/>
@@ -38,4 +39,6 @@
 	<!--with tube maybe more-->
     <xacro:property name="extruder_m" value="1.05"/>
+	<xacro:property name="ee_imu_xyz" value="0 -${(0.035 +(0.0525/2))} 0"/>
+	<xacro:property name="ee_imu_rpy" value="0 3.14159265359 0"/>
 	<xacro:macro name="battery48" params="parent xyz rpy">
 		<xacro:generic_box name="battery48" parent="${parent}" xyz="${xyz}" rpy="${rpy}" dx="${battery_link_dx}" dy="${battery_link_dy}" dz="${battery_link_dz}" m="${battery_link_m}" material="LightGrey" gmaterial="Gazebo/LightGrey" meshfile="battery.dae" mxyz="0.035 0 ${-battery_link_dz/2}" mrpy="0 0 ${M_PI}" />
@@ -87,4 +90,5 @@
 			  <origin xyz= "0 0 ${extruder_h/2}" rpy = "0 0 0" />
 		</joint>
+		<xacro:imu prefix="ee" parent="${parent}" xyz="${ee_imu_xyz}" rpy="${ee_imu_rpy}" />
 	</xacro:macro>
 </robot>

Commit message: armstone base update with compression system

File: as_description/urdf/base/as_base.macro.xacro (robot description, xacro)
@@ -11,14 +11,20 @@
 	<xacro:property name="dc_box_xyz" value=" ${-base_link_dx/2 + 0.02 +dc_box_dy/2} 0 ${base_link_dz/2 - dc_box_dz/2}" />
 	<xacro:property name="dc_box_rpy" value=" 0 0 0" />
-	<xacro:property name="material3_xyz" value="-${base_link_dx/4} 0 ${base_link_dz/2+0.01 + battery_link_dz/2}" />
-	<xacro:property name="material3_rpy" value="0 ${M_PI/2} 0" />
 	<xacro:property name="mount_plate_xyz" value=" ${base_link_dx/2 - mount_plate_dx/2} 0 ${ -base_link_dz/2 +mount_plate_dz/2 +0.02}" />
 	<xacro:property name="mount_plate_rpy" value="0 0 0" />
-	<xacro:property name="compressor_xyz" value="-${base_link_dx/2-compressor_h/2 } ${base_link_dy/2 - compressor_r/2} ${base_link_dz/2-compressor_r }" />
-	<xacro:property name="compressor_rpy" value="0 ${M_PI/2} 0" />
 	<xacro:property name="battery_xyz" value="${-base_link_dx/2 + battery_link_dx/2 -0.08} 0  ${-base_link_dz/2 +0.02 + battery_link_dz/2 }" />
 	<xacro:property name="battery_rpy" value="0 0 0" />
 	<xacro:property name="base_imu_xyz" value="${0.245 +(0.205/2)-(base_link_dx/2)} 0  ${-0.02+base_link_dz/2}" />
 	<xacro:property name="base_imu_rpy" value="0 0 0" />
+	<xacro:property name="compressor_box_xyz" value="${-base_link_dx/2 + compressor_box_dx/2} ${base_link_dy/2 - compressor_box_dy/2 - 0.0713 } ${base_link_dz/2 + compressor_box_dz/2}" />
+	<xacro:property name="compressor_box_rpy" value="0 0 0" />
+	<xacro:property name="material3_xyz" value="${-base_link_dx/2  + 0.235 - material3_h/5} 0 ${base_link_dz/2 + material3_r +0.02}" />
+	<xacro:property name="material3_rpy" value="0 ${M_PI/2} 0" />
+	<xacro:property name="cover_box_xyz" value="${-base_link_dx/2 +cover_box_dx/2} 0 ${base_link_dz/2}" />
+	<xacro:property name="cover_box_rpy" value="0 0 0" />
+	<xacro:property name="ic_box_xyz" value="${-base_link_dx/2  + 0.235 -ic_box_dx/2 + 0.03 } ${-base_link_dy/2 + ic_box_dy/2 +0.04}  ${base_link_dz/2 +ic_box_dz/2}" />
+	<xacro:property name="ic_box_rpy" value="0 0 0" />
+	<xacro:property name="backpack_xyz" value="${-base_link_dx/2  +backpack_dx/2 } 0  ${base_link_dz/2  +backpack_dz/2}" />
+	<xacro:property name="backpack_rpy" value="0 0 0" />
 	<xacro:macro name="as_base" params="load_gazebo_plugin='true'">
 		<!-- Compose the ArmStone Base -->
@@ -28,14 +34,10 @@
 		<xacro:mount_plate parent="base_link" xyz="${mount_plate_xyz}" rpy="${mount_plate_rpy}" />
 		<xacro:imu prefix="base" parent="base_link" xyz="${base_imu_xyz}" rpy="${base_imu_rpy}" />
-		<!-- <xacro:compressor parent="base_link" xyz="${compressor_xyz}" rpy="${compressor_rpy}" /> -->
-		<!-- <xacro:material3 parent="base_link" xyz="${material3_xyz}" rpy="${material3_rpy}" /> -->
-		<!-- gazebo_plugin -->
-		<xacro:if value="${load_gazebo_plugin}">
-			<gazebo>
-				<plugin name="gazebo_ros_control_base" filename="libgazebo_ros_control.so">
-					<robotNamespace>/as_control</robotNamespace>
-				</plugin>
-			</gazebo>
-		</xacro:if>
+		<!--  -->
+		<xacro:compressor parent="base_link" xyz="${compressor_box_xyz}" rpy="${compressor_box_rpy}" />
+		<xacro:material3 parent="base_link" xyz="${material3_xyz}" rpy="${material3_rpy}" />
+		<xacro:cover_plate parent="base_link" xyz="${cover_box_xyz}" rpy="${cover_box_rpy}" />
+		<xacro:ic parent="base_link" xyz="${ic_box_xyz}" rpy="${ic_box_rpy}" />
+		<xacro:backpack parent="base_link" xyz="${backpack_xyz}" rpy="${backpack_rpy}" />
 	</xacro:macro>
 </robot>

File: as_description/urdf/base/components.macro.xacro (robot description, xacro)
@@ -29,8 +29,4 @@
 	<!-- About 3.5 kg aluminium plate. -->
 	<xacro:property name="mount_plate_m" value="${2700*mount_plate_dx*mount_plate_dy*mount_plate_dz}"/>
-	<!-- Compressor -->
-	<xacro:property name="compressor_r" value="0.05"/>
-	<xacro:property name="compressor_h" value="0.13"/>
-	<xacro:property name="compressor_m" value="1.4"/>
 	<!-- Extruder -->
 	<xacro:property name="extruder_r" value="0.05"/>
@@ -54,8 +50,14 @@
 	</xacro:macro>
 	<xacro:macro name="compressor" params="parent xyz rpy">
-		<xacro:generic_cylinder name="compressor" parent="${parent}" xyz="${xyz}" rpy="${rpy}" r="${compressor_r}" h="${compressor_h}" m="${compressor_m}" material="Grey" gmaterial="Gazebo/Grey" meshfile="" mxyz="" mrpy="" />
+		<xacro:generic_box name="compressor" parent="${parent}" xyz="${xyz}" rpy="${rpy}" dx="${compressor_box_dx}" dy="${compressor_box_dy}" dz="${compressor_box_dz}" m="${compressor_m}" material="Grey" gmaterial="Gazebo/Grey" meshfile="compressor_assembly.dae" mxyz="0 0 ${-compressor_box_dz/2}" mrpy="0 0 0" />
 	</xacro:macro>
 	<xacro:macro name="material3" params="parent xyz rpy">
-		<xacro:generic_cylinder name="material3" parent="${parent}" xyz="${xyz}" rpy="${rpy}" r="${material3_r}" h="${material3_h}" m="${material3_m}" material="LightGrey" gmaterial="Gazebo/LightGrey" meshfile="" mxyz="" mrpy=""/>
+		<xacro:generic_cylinder name="material3" parent="${parent}" xyz="${xyz}" rpy="${rpy}" r="${material3_r}" h="${material3_h}" m="${material3_m}" material="LightGrey" gmaterial="Gazebo/LightGrey" meshfile="clay_assembly.dae" mxyz="${material3_r+0.02}  0  ${material3_h/5}" mrpy="0 ${-M_PI/2} 0"/>
+	</xacro:macro>
+	<xacro:macro name="cover_plate" params="parent xyz rpy">
+		<xacro:generic_box name="cover_plate" parent="${parent}" xyz="${xyz}" rpy="${rpy}" dx="${cover_box_dx}" dy="${cover_box_dy}" dz="${cover_box_dz}" m="${cover_plate_m}" material="LightGrey" gmaterial="Gazebo/LightGrey" meshfile="cover_assembly_.dae" mxyz="0 0 0" mrpy="0 0 0"/>
+	</xacro:macro>
+	<xacro:macro name="ic" params="parent xyz rpy">
+		<xacro:generic_box name="ic" parent="${parent}" xyz="${xyz}" rpy="${rpy}" dx="${ic_box_dx}" dy="${ic_box_dy}" dz="${ic_box_dz}" m="${ic_m}" material="LightGrey" gmaterial="Gazebo/LightGrey" meshfile="intermediate_assembly.dae" mxyz="${ic_box_dx/2 - 0.03} 0 ${-ic_box_dz/2}" mrpy="0 0 0"/>
 	</xacro:macro>
 	<xacro:macro name="extruder" params="parent xyz rpy">
@@ -92,3 +94,17 @@
 		<xacro:imu prefix="ee" parent="${parent}" xyz="${ee_imu_xyz}" rpy="${ee_imu_rpy}" />
 	</xacro:macro>
+	<xacro:macro name="backpack" params="parent xyz rpy">
+		<joint name="backpack_joint" type="fixed">
+            <parent link="${parent}"/>
+            <child link="backpack_link"/>
+            <origin xyz= "${xyz}" rpy = "${rpy}" />
+        </joint>
+        <link name="backpack_link">
+			<collision>
+                <geometry>
+                    <box size="${backpack_dx} ${backpack_dy} ${backpack_dz}" />
+                </geometry>
+            </collision>
+        </link>
+	</xacro:macro>
 </robot>

File: as_description/urdf/base/components.params.xacro (robot description, xacro)
@@ -17,8 +17,4 @@
 	<xacro:property name="dc_box_dz" value="0.068"/>
 	<xacro:property name="dc_box_m" value="1.8"/>
-	<!-- Material Cylinder 3 -->
-	<xacro:property name="material3_r" value="0.0525"/>
-	<xacro:property name="material3_h" value="0.42"/>
-	<xacro:property name="material3_m" value="${3*1760/1000}"/>
 	<!-- Aluminium plate -->
 	<xacro:property name="mount_plate_dx" value="${0.72/2}"/>
@@ -29,6 +25,25 @@
 	<xacro:property name="mount_plate_m" value="${2700*mount_plate_dx*mount_plate_dy*mount_plate_dz}"/>
 	<!-- Compressor -->
-	<xacro:property name="compressor_r" value="0.05"/>
-	<xacro:property name="compressor_h" value="0.13"/>
-	<xacro:property name="compressor_m" value="1.4"/>
+	<xacro:property name="compressor_box_dx" value="0.242"/>
+	<xacro:property name="compressor_box_dy" value="0.055"/>
+	<xacro:property name="compressor_box_dz" value="0.12"/>
+	<xacro:property name="compressor_m" value="1.1"/>
+	<!-- Material Cylinder 3 -->
+	<xacro:property name="material3_r" value="${0.2/2}"/>
+	<xacro:property name="material3_h" value="0.5"/>
+	<xacro:property name="material3_m" value="${3*1760/1000}"/>
+	<!-- Compressor -->
+	<xacro:property name="cover_box_dx" value="0.47"/>
+	<xacro:property name="cover_box_dy" value="0.45"/>
+	<xacro:property name="cover_box_dz" value="0.006"/>
+	<xacro:property name="cover_plate_m" value="0.2"/>
+	<!-- Compressor -->
+	<xacro:property name="ic_box_dx" value="0.28"/>
+	<xacro:property name="ic_box_dy" value="0.074"/>
+	<xacro:property name="ic_box_dz" value="0.145"/>
+	<xacro:property name="ic_m" value="0.4"/>
+	<!-- backpack -->
+	<xacro:property name="backpack_dx" value="0.4"/>
+	<xacro:property name="backpack_dy" value="0.4"/>
+	<xacro:property name="backpack_dz" value="0.18"/>
 </robot>

Commit message: (no branch):wip  sensors gazebo

File: as_description/urdf/base/as_base.macro.xacro (robot description, xacro)
@@ -27,4 +27,8 @@
 	<xacro:property name="backpack_xyz" value="${-base_link_dx/2  +backpack_dx/2 } 0  ${base_link_dz/2  +backpack_dz/2}" />
 	<xacro:property name="backpack_rpy" value="0 0 0" />
+	<xacro:property name="left_hokuyo_xyz" value="${-base_link_dx/2 + 0.235} ${base_link_dy/2 - 0.02 }  0" />
+	<xacro:property name="left_hokuyo_rpy" value="0 0 ${M_PI/2}" />
+	<xacro:property name="right_hokuyo_xyz" value="${-base_link_dx/2 + 0.235} ${-base_link_dy/2  + 0.02 }  0" />
+	<xacro:property name="right_hokuyo_rpy" value="0 0 ${- M_PI/2}" />
 	<xacro:macro name="as_base" params="load_gazebo_plugin='true'">
 		<!-- Compose the ArmStone Base -->
@@ -33,6 +37,5 @@
 		<xacro:dc_box parent="base_link" xyz="${dc_box_xyz}" rpy="${dc_box_rpy}" />
 		<xacro:mount_plate parent="base_link" xyz="${mount_plate_xyz}" rpy="${mount_plate_rpy}" />
-		<xacro:imu prefix="base" parent="base_link" xyz="${base_imu_xyz}" rpy="${base_imu_rpy}" />
-		<!--  -->
+		<!-- Attachements -->
 		<xacro:compressor parent="base_link" xyz="${compressor_box_xyz}" rpy="${compressor_box_rpy}" />
 		<xacro:material3 parent="base_link" xyz="${material3_xyz}" rpy="${material3_rpy}" />
@@ -40,4 +43,8 @@
 		<xacro:ic parent="base_link" xyz="${ic_box_xyz}" rpy="${ic_box_rpy}" />
 		<xacro:backpack parent="base_link" xyz="${backpack_xyz}" rpy="${backpack_rpy}" />
+		<!-- Sensors -->
+		<xacro:imu prefix="base" parent="base_link" xyz="${base_imu_xyz}" rpy="${base_imu_rpy}" />
+		<xacro:hokuyo prefix="left" parent="base_link" xyz="${left_hokuyo_xyz}" rpy="${left_hokuyo_rpy}" />
+		<xacro:hokuyo prefix="right" parent="base_link" xyz="${right_hokuyo_xyz}" rpy="${right_hokuyo_rpy}" />
 	</xacro:macro>
 </robot>

File: as_description/urdf/base/components.macro.xacro (robot description, xacro)
@@ -106,3 +106,60 @@
         </link>
 	</xacro:macro>
+	<xacro:macro name="hokuyo" params="parent xyz rpy prefix">
+		<joint name="${prefix}_hokuyo_joint" type="fixed">
+            <parent link="${parent}"/>
+            <child link="${prefix}_hokuyo_link"/>
+            <origin xyz= "${xyz}" rpy = "${rpy}" />
+        </joint>
+        <link name="${prefix}_hokuyo_link">
+			<inertial>
+				<mass value="1e-5" />
+				<origin xyz="0 0 0" rpy="0 0 0"/>
+				<inertia ixx="1e-6" ixy="0" ixz="0" iyy="1e-6" iyz="0" izz="1e-6" />
+			</inertial>
+			<visual>
+				<origin xyz="0.0484 0 0" rpy="0 0 ${M_PI/2}"/>
+				<geometry>
+					<mesh filename="package://as_description/meshes/hokuyo${mesh_filetype}"/>
+				</geometry>
+			</visual>
+        </link>
+		<gazebo reference="${prefix}_hokuyo_link">
+			<!-- <sensor type="gpu_ray" name="${prefix}_hokuyo_sensor"> -->
+			<sensor type="ray" name="${prefix}_hokuyo_sensor">
+				<pose>0 0 0 0 0 0</pose>
+				<visualize>true</visualize>
+				<update_rate>10</update_rate>
+				<ray>
+					<scan>
+						<horizontal>
+							<samples>683</samples>
+							<resolution>1</resolution>
+							<min_angle>-2.09439510239</min_angle>
+							<max_angle>2.09439510239</max_angle>
+						</horizontal>
+					</scan>
+					<range>
+						<min>0.10</min>
+						<max>4.0</max>
+						<resolution>0.001</resolution>
+					</range>
+					<noise>
+						<type>gaussian</type>
+						<!-- Noise parameters based on published spec for Hokuyo laser
+							achieving "+-30mm" accuracy at range < 10m.  A mean of 0.0m and
+							stddev of 0.01m will put 99.7% of samples within 0.03m of the true
+							reading. -->
+						<mean>0.0</mean>
+						<stddev>0.015</stddev>
+					</noise>
+				</ray>
+				<!-- <plugin name="${prefix}_hokuyo_gazebo_driver" filename="libgazebo_ros_gpu_laser.so"> -->
+				<plugin name="${prefix}_hokuyo_gazebo_driver" filename="libgazebo_ros_laser.so">
+					<topicName>/as_localisation/scan</topicName>
+					<frameName>${prefix}_hokuyo_link</frameName>
+				</plugin>
+			</sensor>
+		</gazebo>
+	</xacro:macro>
 </robot>
