Commit message: minor urdfs

File: as_description/urdf/base/components.macro.xacro (robot description, xacro)
@@ -20,8 +20,4 @@
 	<xacro:property name="dc_box_dz" value="0.068"/>
 	<xacro:property name="dc_box_m" value="1.8"/>
-	<!-- Material Cylinder 3 -->
-	<xacro:property name="material3_r" value="0.0525"/>
-	<xacro:property name="material3_h" value="0.42"/>
-	<xacro:property name="material3_m" value="${3*1760/1000}"/>
 	<!-- Aluminium plate -->
 	<xacro:property name="mount_plate_dx" value="${0.27}"/>

File: as_description/urdf/base/components.params.xacro (robot description, xacro)
@@ -32,15 +32,15 @@
 	<xacro:property name="material3_r" value="${0.2/2}"/>
 	<xacro:property name="material3_h" value="0.5"/>
-	<xacro:property name="material3_m" value="${3*1760/1000}"/>
+	<xacro:property name="material3_m" value="${1.75 + 3*1760/1000}"/>
 	<!-- Compressor -->
 	<xacro:property name="cover_box_dx" value="0.47"/>
 	<xacro:property name="cover_box_dy" value="0.45"/>
 	<xacro:property name="cover_box_dz" value="0.006"/>
-	<xacro:property name="cover_plate_m" value="0.2"/>
+	<xacro:property name="cover_plate_m" value="1.45"/>
 	<!-- Compressor -->
 	<xacro:property name="ic_box_dx" value="0.28"/>
 	<xacro:property name="ic_box_dy" value="0.074"/>
 	<xacro:property name="ic_box_dz" value="0.145"/>
-	<xacro:property name="ic_m" value="0.4"/>
+	<xacro:property name="ic_m" value="0.83"/>
 	<!-- backpack -->
 	<xacro:property name="backpack_dx" value="0.4"/>

Commit message: wip slam

File: as_description/urdf/base/components.macro.xacro (robot description, xacro)
@@ -3,4 +3,5 @@
 	<xacro:include filename="$(find as_description)/urdf/common/generic_links.xacro"/>
 	<xacro:include filename="$(find sensor_imu)/urdf/sensor_imu.xacro"/>
+	<xacro:include filename="$(find realsense2_description)/urdf/_l515.urdf.xacro" />
 	<xacro:property name="mesh_filetype" value=".dae" />
 	<!-- <xacro:property name="mesh_filetype" value=".stl" /> -->
@@ -59,5 +60,5 @@
 		<xacro:generic_box name="ic" parent="${parent}" xyz="${xyz}" rpy="${rpy}" dx="${ic_box_dx}" dy="${ic_box_dy}" dz="${ic_box_dz}" m="${ic_m}" material="LightGrey" gmaterial="Gazebo/LightGrey" meshfile="intermediate_assembly${mesh_filetype}" mxyz="${ic_box_dx/2 - 0.03} 0 ${-ic_box_dz/2}" mrpy="0 0 0"/>
 	</xacro:macro>
-	<xacro:macro name="extruder" params="parent xyz rpy">
+	<xacro:macro name="extruder" params="parent xyz rpy l515l_on:=true">
 		<joint name="extruder_joint" type="fixed">
             <parent link="${parent}"/>
@@ -91,4 +92,34 @@
 		</joint>
 		<xacro:imu prefix="ee" parent="${parent}" xyz="${ee_imu_xyz}" rpy="${ee_imu_rpy}" />
+		<xacro:if value="${l515l_on}">
+			<joint name="cam_holder_joint" type="fixed">
+				<parent link="extruder_ee"/>
+				<child link="cam_holder_link"/>
+				<origin xyz= "-0.056217 0 -0.170" rpy = "0 0 ${M_PI}" />
+			</joint>
+			<link name="cam_holder_link">
+				<visual>
+					<origin xyz= "0 0 0" rpy = "0 0 0" />
+					<geometry>
+						<mesh filename="package://as_description/meshes/cam_holder${mesh_filetype}" />
+					</geometry>
+				</visual>
+				<collision>
+					<origin xyz= "0 0 0" rpy = "0 0 0" />
+					<geometry>
+						<mesh filename="package://as_description/meshes/cam_holder${mesh_filetype}" />
+					</geometry>
+				</collision>
+			</link>
+			<joint name="cam_holder_offest_joint" type="fixed">
+				<parent link="cam_holder_link"/>
+				<child link="cam_holder_end_link"/>
+				<origin xyz= "0.1264 0 -0.1244" rpy = "${-25*M_PI/180} 0  ${M_PI/2}" />
+			</joint>
+			<link name="cam_holder_end_link"/>
+			<xacro:sensor_l515 name="l515" topics_ns="/as_sensors/depth_cam" parent="cam_holder_end_link" use_nominal_extrinsics="true" publish_pointcloud="true" add_plug="false" use_mesh="true">
+				<origin xyz="0.0305 0  0.011057" rpy="0 ${-90*M_PI/180} 0" />
+			</xacro:sensor_l515>
+		</xacro:if>
 	</xacro:macro>
 	<xacro:macro name="backpack" params="parent xyz rpy">
@@ -157,5 +188,5 @@
 				<!-- <plugin name="${prefix}_hokuyo_gazebo_driver" filename="libgazebo_ros_gpu_laser.so"> -->
 				<plugin name="${prefix}_hokuyo_gazebo_driver" filename="libgazebo_ros_laser.so">
-					<topicName>/as_localisation/scan</topicName>
+					<topicName>/as_sensors/scan</topicName>
 					<frameName>${prefix}_hokuyo_link</frameName>
 				</plugin>

Commit message: wip_slam toolbox

File: as_description/urdf/base/components.macro.xacro (robot description, xacro)
@@ -156,5 +156,11 @@
 			</visual>
         </link>
-		<gazebo reference="${prefix}_hokuyo_link">
+		<joint name="${prefix}_hokuyo_joint2" type="fixed">
+            <parent link="${prefix}_hokuyo_link"/>
+            <child link="${prefix}_hokuyo_laser"/>
+            <origin xyz= "0.02 0 0.04" rpy = "0 0 0" />
+        </joint>
+		<link name="${prefix}_hokuyo_laser"/>
+		<gazebo reference="${prefix}_hokuyo_laser">
 			<!-- <sensor type="gpu_ray" name="${prefix}_hokuyo_sensor"> -->
 			<sensor type="ray" name="${prefix}_hokuyo_sensor">

Commit message: wip

File: as_description/urdf/base/components.macro.xacro (robot description, xacro)
@@ -60,5 +60,5 @@
 		<xacro:generic_box name="ic" parent="${parent}" xyz="${xyz}" rpy="${rpy}" dx="${ic_box_dx}" dy="${ic_box_dy}" dz="${ic_box_dz}" m="${ic_m}" material="LightGrey" gmaterial="Gazebo/LightGrey" meshfile="intermediate_assembly${mesh_filetype}" mxyz="${ic_box_dx/2 - 0.03} 0 ${-ic_box_dz/2}" mrpy="0 0 0" />
 	</xacro:macro>
-	<xacro:macro name="extruder" params="parent xyz rpy l515l_on:=true">
+	<xacro:macro name="extruder" params="parent xyz rpy">
 		<joint name="extruder_joint" type="fixed">
 			<parent link="${parent}" />
@@ -85,5 +85,4 @@
 			</collision>
 		</link>
-		<link name="extruder_ee" />
 		<joint name="extruder_ee_joint" type="fixed">
 			<parent link="extruder_link" />
@@ -91,35 +90,84 @@
 			<origin xyz="0 0 ${extruder_h/2}" rpy="0 0 0" />
 		</joint>
+		<link name="extruder_ee" />
 		<xacro:imu prefix="ee" parent="${parent}" xyz="${ee_imu_xyz}" rpy="${ee_imu_rpy}" />
-		<xacro:if value="${l515l_on}">
-			<joint name="cam_holder_joint" type="fixed">
-				<parent link="extruder_ee" />
-				<child link="cam_holder_link" />
-				<origin xyz="-0.056217 0 -0.170" rpy="0 0 ${M_PI}" />
-			</joint>
-			<link name="cam_holder_link">
-				<visual>
-					<origin xyz="0 0 0" rpy="0 0 0" />
-					<geometry>
-						<mesh filename="package://as_description/meshes/cam_holder${mesh_filetype}" />
-					</geometry>
-				</visual>
-				<collision>
-					<origin xyz="0 0 0" rpy="0 0 0" />
-					<geometry>
-						<mesh filename="package://as_description/meshes/cam_holder${mesh_filetype}" />
-					</geometry>
-				</collision>
-			</link>
-			<joint name="cam_holder_offest_joint" type="fixed">
-				<parent link="cam_holder_link" />
-				<child link="cam_holder_end_link" />
-				<origin xyz="0.1264 0 -0.1244" rpy="${-25*M_PI/180} 0  ${M_PI/2}" />
-			</joint>
-			<link name="cam_holder_end_link" />
-			<xacro:sensor_l515 name="l515" topics_ns="/as_sensors/depth_cam" parent="cam_holder_end_link" use_nominal_extrinsics="true" publish_pointcloud="true" add_plug="false" use_mesh="true">
-				<origin xyz="0.0305 0  0.011057" rpy="0 ${-90*M_PI/180} 0" />
-			</xacro:sensor_l515>
-		</xacro:if>
+		<!-- Extruder Axes -->
+		<joint name="extruder_axes_joint" type="fixed">
+			<parent link="${parent}" />
+			<child link="extruder_axes_link" />
+			<origin xyz="0.038884 -0.018177 -0.001" rpy="0 ${M_PI} ${M_PI}" />
+		</joint>
+		<link name="extruder_axes_link">
+			<visual>
+				<origin xyz="0 0 0" rpy="0 0 0" />
+				<geometry>
+					<mesh filename="package://as_description/meshes/extruder_axes${mesh_filetype}" />
+				</geometry>
+			</visual>
+			<collision>
+				<origin xyz="0 0 0" rpy="0 0 0" />
+				<geometry>
+					<mesh filename="package://as_description/meshes/extruder_axes${mesh_filetype}" />
+				</geometry>
+			</collision>
+		</link>
+		<!-- LEFT is D435 -->
+		<joint name="d435_holder_joint" type="fixed">
+			<parent link="${parent}" />
+			<child link="d435_holder_link" />
+			<origin xyz="0 0.056202 -0.001" rpy="0 0 ${M_PI/2}" />
+		</joint>
+		<link name="d435_holder_link">
+			<visual>
+				<origin xyz="0 0 0" rpy="0 0 0" />
+				<geometry>
+					<mesh filename="package://as_description/meshes/cam_holder${mesh_filetype}" />
+				</geometry>
+			</visual>
+			<collision>
+				<origin xyz="0 0 0" rpy="0 0 0" />
+				<geometry>
+					<mesh filename="package://as_description/meshes/cam_holder${mesh_filetype}" />
+				</geometry>
+			</collision>
+		</link>
+		<joint name="d435_mount_joint" type="fixed">
+			<parent link="d435_holder_link" />
+			<child link="d435_mount_link" />
+			<origin xyz="0.1264 0 -0.1244" rpy="${-25*M_PI/180} 0  ${M_PI/2}" />
+		</joint>
+		<link name="d435_mount_link" />
+		<!-- RIGHT is realsense -->
+		<joint name="l515_holder_joint" type="fixed">
+			<parent link="${parent}" />
+			<child link="l515_holder_link" />
+			<origin xyz="0 -0.056202 -0.001" rpy="0 0 ${-M_PI/2}" />
+		</joint>
+		<link name="l515_holder_link">
+			<visual>
+				<origin xyz="0 0 0" rpy="0 0 0" />
+				<geometry>
+					<mesh filename="package://as_description/meshes/cam_holder${mesh_filetype}" />
+				</geometry>
+			</visual>
+			<collision>
+				<origin xyz="0 0 0" rpy="0 0 0" />
+				<geometry>
+					<mesh filename="package://as_description/meshes/cam_holder${mesh_filetype}" />
+				</geometry>
+			</collision>
+		</link>
+		<joint name="l515_mount_joint" type="fixed">
+			<parent link="l515_holder_link" />
+			<child link="l515_mount_link" />
+			<origin xyz="0.1264 0 -0.1244" rpy="${-25*M_PI/180} 0  ${M_PI/2}" />
+		</joint>
+		<link name="l515_mount_link" />
+		<xacro:sensor_l515 name="l515" topics_ns="/as_sensors/l515/depth_cam" parent="l515_mount_link" use_nominal_extrinsics="true" publish_pointcloud="true" add_plug="false" use_mesh="true">
+			<origin xyz="0.0305 0  0.011057" rpy="0 ${-90*M_PI/180} 0" />
+		</xacro:sensor_l515>
+		<!-- <xacro:sensor_l515 name="l515" topics_ns="/as_sensors/d435/depth_cam" parent="d435_mount_link" use_nominal_extrinsics="true" publish_pointcloud="true" add_plug="false" use_mesh="true">
+			<origin xyz="0.0305 0  0.011057" rpy="0 ${-90*M_PI/180} 0" />
+		</xacro:sensor_l515> -->
 	</xacro:macro>
 	<xacro:macro name="backpack" params="parent xyz rpy">

Commit message: Messing artound with dae and setting the lcamera links properly

File: as_description/urdf/base/components.macro.xacro (robot description, xacro)
@@ -3,5 +3,6 @@
 	<xacro:include filename="$(find as_description)/urdf/common/generic_links.xacro" />
 	<xacro:include filename="$(find sensor_imu)/urdf/sensor_imu.xacro" />
-	<xacro:include filename="$(find realsense2_description)/urdf/_l515.urdf.xacro" />
+	<xacro:include filename="$(find as_description)/urdf/components/_l515.urdf.xacro" />
+	<!-- <xacro:include filename="$(find realsense2_description)/urdf/_d435.urdf.xacro" /> -->
 	<xacro:property name="mesh_filetype" value=".dae" />
 	<!-- <xacro:property name="mesh_filetype" value=".stl" /> -->
@@ -96,5 +97,5 @@
 			<parent link="${parent}" />
 			<child link="extruder_axes_link" />
-			<origin xyz="0.038884 -0.018177 -0.001" rpy="0 ${M_PI} ${M_PI}" />
+			<origin xyz="0.018177 0.038884 -0.001" rpy="0 ${M_PI} ${-M_PI/2}" />
 		</joint>
 		<link name="extruder_axes_link">
@@ -116,5 +117,5 @@
 			<parent link="${parent}" />
 			<child link="d435_holder_link" />
-			<origin xyz="0 0.056202 -0.001" rpy="0 0 ${M_PI/2}" />
+			<origin xyz="0.056202 0  -0.001" rpy="0 0 0" />
 		</joint>
 		<link name="d435_holder_link">
@@ -135,5 +136,5 @@
 			<parent link="d435_holder_link" />
 			<child link="d435_mount_link" />
-			<origin xyz="0.1264 0 -0.1244" rpy="${-25*M_PI/180} 0  ${M_PI/2}" />
+			<origin xyz="0.156687 0 -0.1207278" rpy="${-30*M_PI/180} 0  ${M_PI/2}" />
 		</joint>
 		<link name="d435_mount_link" />
@@ -142,5 +143,5 @@
 			<parent link="${parent}" />
 			<child link="l515_holder_link" />
-			<origin xyz="0 -0.056202 -0.001" rpy="0 0 ${-M_PI/2}" />
+			<origin xyz="-0.056202 0  -0.001" rpy="0 0 ${M_PI}" />
 		</joint>
 		<link name="l515_holder_link">
@@ -161,13 +162,18 @@
 			<parent link="l515_holder_link" />
 			<child link="l515_mount_link" />
-			<origin xyz="0.1264 0 -0.1244" rpy="${-25*M_PI/180} 0  ${M_PI/2}" />
+			<origin xyz="0.16113414 0.02 -0.11987969" rpy="${-30*M_PI/180} 0  ${M_PI/2}" />
+			<!-- -161.13414
+			119.87969
+			+-20.00000 -->
 		</joint>
 		<link name="l515_mount_link" />
-		<xacro:sensor_l515 name="l515" topics_ns="/as_sensors/l515/depth_cam" parent="l515_mount_link" use_nominal_extrinsics="true" publish_pointcloud="true" add_plug="false" use_mesh="true">
-			<origin xyz="0.0305 0  0.011057" rpy="0 ${-90*M_PI/180} 0" />
+		<xacro:sensor_l515 name="l515_mount_link" topics_ns="/as_sensors/l515/depth_cam" parent="l515_mount_link" use_nominal_extrinsics="true" publish_pointcloud="true" add_plug="false" use_mesh="true">
+			<origin xyz="0.01015 0  0.014" rpy="0 ${-M_PI/2} 0" />
+			<!-- From starting frame to screw hole closer to usb-c: -0.014;0;0.01015 -->
+			<!-- From starting frame to screw hole further to usb-c: -0.014;0;0.05015 -->
 		</xacro:sensor_l515>
-		<!-- <xacro:sensor_l515 name="l515" topics_ns="/as_sensors/d435/depth_cam" parent="d435_mount_link" use_nominal_extrinsics="true" publish_pointcloud="true" add_plug="false" use_mesh="true">
-			<origin xyz="0.0305 0  0.011057" rpy="0 ${-90*M_PI/180} 0" />
-		</xacro:sensor_l515> -->
+		<!-- <xacro:sensor_d435 parent="d435_mount_link" use_nominal_extrinsics="true" add_plug="false" use_mesh="true">
+			<origin xyz="0 0 0" rpy="0 0 0"/>
+		</xacro:sensor_d435> -->
 	</xacro:macro>
 	<xacro:macro name="backpack" params="parent xyz rpy">

Commit message: WIP

File: as_description/urdf/base/components.macro.xacro (robot description, xacro)
@@ -34,5 +34,6 @@
 	<!--Without material m 1.05 (including bolts)  -->
 	<!--with tube maybe more-->
-	<xacro:property name="extruder_m" value="1.05" />
+	<!-- measured jan 16: 751+800 -->
+	<xacro:property name="extruder_m" value="1.75" />
 	<xacro:property name="ee_imu_xyz" value="0 -${(0.035 +(0.0525/2))} 0" />
 	<xacro:property name="ee_imu_rpy" value="0 3.14159265359 0" />

Commit message: wip

File: as_description/urdf/base/components.macro.xacro (robot description, xacro)
@@ -171,11 +171,11 @@
 		</joint>
 		<link name="l515_mount_link" />
-		<xacro:if value="${load_sensors}">
+		<!-- <xacro:if value="${load_sensors}">
 			<xacro:sensor_l515 name="l515_mount_link" topics_ns="/as_sensors/l515/depth_cam" parent="l515_mount_link" use_nominal_extrinsics="true" publish_pointcloud="true" add_plug="false" use_mesh="true">
-			<origin xyz="0.01015 0  0.014" rpy="0 ${-M_PI/2} 0" />
+			<origin xyz="0.01015 0  0.014" rpy="0 ${-M_PI/2} 0" /> -->
 			<!-- From starting frame to screw hole closer to usb-c: -0.014;0;0.01015 -->
 			<!-- From starting frame to screw hole further to usb-c: -0.014;0;0.05015 -->
-			</xacro:sensor_l515>
-		</xacro:if>
+			<!-- </xacro:sensor_l515> -->
+		<!-- </xacro:if> -->
 		<!-- <xacro:sensor_d435 parent="d435_mount_link" use_nominal_extrinsics="true" add_plug="false" use_mesh="true">
 			<origin xyz="0 0 0" rpy="0 0 0"/>
